File: tempmux.sch (KiCad schematic (older format))
At the start: 0 parts

Commit message: Finished Temp Sheet
Parts:
- added C?: 0.1uF, symbol Device:C_Small
- added J?: Conn_02x07_Counter_Clockwise, symbol Connector_Generic:Conn_02x07_Counter_Clockwise
- added R? (x12): 22k, symbol Device:R
- added U?: CD74HC4067SM, Package_SO:SSOP-24_5.3x8.2mm_P0.65mm, symbol 74xx:CD74HC4067SM
Connections:
- new net +5V: C?.1, J?.1 (Pin_1), J?.14 (Pin_14), U?.24 (VCC)
- new net COM: U?.1 (COM)
- new net CellTemp_1: J?.2 (Pin_2), R?.1, U?.9 (I0)
- new net CellTemp_10: J?.11 (Pin_11), R?.1, U?.22 (I9)
- new net CellTemp_11: J?.12 (Pin_12), R?.1, U?.21 (I10)
- new net CellTemp_12: J?.13 (Pin_13), R?.1, U?.20 (I11)
- new net CellTemp_2: J?.3 (Pin_3), R?.1, U?.8 (I1)
- new net CellTemp_3: J?.4 (Pin_4), R?.1, U?.7 (I2)
- new net CellTemp_4: J?.5 (Pin_5), R?.1, U?.6 (I3)
- new net CellTemp_5: J?.6 (Pin_6), R?.1, U?.5 (I4)
- new net CellTemp_6: J?.7 (Pin_7), R?.1, U?.4 (I5)
- new net CellTemp_7: J?.8 (Pin_8), R?.1, U?.3 (I6)
- new net CellTemp_8: J?.9 (Pin_9), R?.1, U?.2 (I7)
- new net CellTemp_9: J?.10 (Pin_10), R?.1, U?.23 (I8)
- new net GND: C?.2, R?.2, R?.2, R?.2, R?.2, R?.2, R?.2, R?.2, R?.2, R?.2, R?.2, R?.2, R?.2, U?.12 (GND), U?.16 (I15), U?.17 (I14), U?.18 (I13), U?.19 (I12)
- new net S0: U?.10 (S0)
- new net S1: U?.11 (S1)
- new net S2: U?.14 (S2)
- new net S3: U?.13 (S3)
- new net ~Enable~: U?.15 (~E)
Other:
- note added: "* Through resistance of Analogue Mux is around 60\n Ohms and connects to ADC\n which has input impedence of about 10M Ohm"

Commit message: Think I just added labels?
Parts:
- gave numbers to parts that had none: 15
Changed lines of the file:
@@
 P 2000 2200
 AR Path="/5F70A721/5F6868D3" Ref="U?"  Part="1"
-AR Path="/5F70B1A3/5F6868D3" Ref="U?"  Part="1"
-F 0 "U?" H 2000 2200 50  0000 C CNN
+AR Path="/5F70B1A3/5F6868D3" Ref="U12"  Part="1"
+F 0 "U12" H 2000 2200 50  0000 C CNN
 F 1 "CD74HC4067SM" H 1600 3100 50  0000 C CNN
 F 2 "Package_SO:SSOP-24_5.3x8.2mm_P0.65mm" H 3050 1200 50  0001 C CIN
@@
 P 2000 3400
 AR Path="/5F70A721/5F6868D9" Ref="#PWR?"  Part="1"
-AR Path="/5F70B1A3/5F6868D9" Ref="#PWR?"  Part="1"
-F 0 "#PWR?" H 2000 3150 50  0001 C CNN
+AR Path="/5F70B1A3/5F6868D9" Ref="#PWR0153"  Part="1"
+F 0 "#PWR0153" H 2000 3150 50  0001 C CNN
 F 1 "GND" H 2005 3227 50  0000 C CNN
 F 2 "" H 2000 3400 50  0001 C CNN
@@
 P 2150 1100
 AR Path="/5F70A721/5F6868E0" Ref="C?"  Part="1"
-AR Path="/5F70B1A3/5F6868E0" Ref="C?"  Part="1"
-F 0 "C?" H 2242 1146 50  0000 L CNN
+AR Path="/5F70B1A3/5F6868E0" Ref="C12"  Part="1"
+F 0 "C12" H 2242 1146 50  0000 L CNN
 F 1 "0.1uF" H 2242 1055 50  0000 L CNN
 F 2 "" H 2150 1100 50  0001 C CNN
@@
 P 2150 1200
 AR Path="/5F70A721/5F6868E6" Ref="#PWR?"  Part="1"
-AR Path="/5F70B1A3/5F6868E6" Ref="#PWR?"  Part="1"
-F 0 "#PWR?" H 2150 950 50  0001 C CNN
+AR Path="/5F70B1A3/5F6868E6" Ref="#PWR0154"  Part="1"
+F 0 "#PWR0154" H 2150 950 50  0001 C CNN
 F 1 "GND" H 2300 1150 50  0000 C CNN
 F 2 "" H 2150 1200 50  0001 C CNN
@@
 P 2000 950
 AR Path="/5F70A721/5F6868EC" Ref="#PWR?"  Part="1"
-AR Path="/5F70B1A3/5F6868EC" Ref="#PWR?"  Part="1"
-F 0 "#PWR?" H 2000 800 50  0001 C CNN
+AR Path="/5F70B1A3/5F6868EC" Ref="#PWR0155"  Part="1"
+F 0 "#PWR0155" H 2000 800 50  0001 C CNN
 F 1 "+5V" H 2015 1123 50  0000 C CNN
 F 2 "" H 2000 950 50  0001 C CNN
@@
 P 9900 1850
 AR Path="/5F70A721/5F68B135" Ref="J?"  Part="1"
-AR Path="/5F70B1A3/5F68B135" Ref="J?"  Part="1"
-F 0 "J?" H 9950 2300 50  0000 C CNN
+AR Path="/5F70B1A3/5F68B135" Ref="J2"  Part="1"
+F 0 "J2" H 9950 2300 50  0000 C CNN
 F 1 "Conn_02x07_Counter_Clockwise" H 9950 1450 50  0000 C CNN
 F 2 "" H 9900 1850 50  0001 C CNN
@@
 P 9650 1550
 AR Path="/5F70A721/5F68DF75" Ref="#PWR?"  Part="1"
-AR Path="/5F70B1A3/5F68DF75" Ref="#PWR?"  Part="1"
-F 0 "#PWR?" H 9650 1400 50  0001 C CNN
+AR Path="/5F70B1A3/5F68DF75" Ref="#PWR0156"  Part="1"
+F 0 "#PWR0156" H 9650 1400 50  0001 C CNN
 F 1 "+5V" H 9665 1723 50  0000 C CNN
 F 2 "" H 9650 1550 50  0001 C CNN
@@
 P 10250 1550
 AR Path="/5F70A721/5F68E7C7" Ref="#PWR?"  Part="1"
-AR Path="/5F70B1A3/5F68E7C7" Ref="#PWR?"  Part="1"
-F 0 "#PWR?" H 10250 1400 50  0001 C CNN
+AR Path="/5F70B1A3/5F68E7C7" Ref="#PWR0157"  Part="1"
+F 0 "#PWR0157" H 10250 1400 50  0001 C CNN
 F 1 "+5V" H 10265 1723 50  0000 C CNN
 F 2 "" H 10250 1550 50  0001 C CNN
@@
 	10200 1650 10300 1650
 $Comp
-L Device:R R?
+L Device:R R58
 U 1 1 5F69A862
 P 5000 1650
-F 0 "R?" H 5070 1696 50  0000 L CNN
+F 0 "R58" H 5070 1696 50  0000 L CNN
 F 1 "22k" H 5070 1605 50  0000 L CNN
 F 2 "" V 4930 1650 50  0001 C CNN
@@
 $EndComp
 $Comp
-L Device:R R?
+L Device:R R60
 U 1 1 5F69AE56
 P 5500 1650
-F 0 "R?" H 5570 1696 50  0000 L CNN
+F 0 "R60" H 5570 1696 50  0000 L CNN
 F 1 "22k" H 5570 1605 50  0000 L CNN
 F 2 "" V 5430 1650 50  0001 C CNN
@@
 $EndComp
 $Comp
-L Device:R R?
+L Device:R R62
 U 1 1 5F69AFF2
 P 6000 1650
-F 0 "R?" H 6070 1696 50  0000 L CNN
+F 0 "R62" H 6070 1696 50  0000 L CNN
 F 1 "22k" H 6070 1605 50  0000 L CNN
 F 2 "" V 5930 1650 50  0001 C CNN
@@
 $EndComp
 $Comp
-L Device:R R?
+L Device:R R64
 U 1 1 5F69B1F7
 P 6500 1650
-F 0 "R?" H 6570 1696 50  0000 L CNN
+F 0 "R64" H 6570 1696 50  0000 L CNN
 F 1 "22k" H 6570 1605 50  0000 L CNN
 F 2 "" V 6430 1650 50  0001 C CNN
@@
 $EndComp
 $Comp
-L Device:R R?
+L Device:R R66
 U 1 1 5F69B4CD
 P 7000 1650
-F 0 "R?" H 7070 1696 50  0000 L CNN
+F 0 "R66" H 7070 1696 50  0000 L CNN
 F 1 "22k" H 7070 1605 50  0000 L CNN
 F 2 "" V 6930 1650 50  0001 C CNN
@@
 $EndComp
 $Comp
-L Device:R R?
+L Device:R R68
 U 1 1 5F69B7DC
 P 7500 1650
-F 0 "R?" H 7570 1696 50  0000 L CNN
+F 0 "R68" H 7570 1696 50  0000 L CNN
 F 1 "22k" H 7570 1605 50  0000 L CNN
 F 2 "" V 7430 1650 50  0001 C CNN
@@
 $EndComp
 $Comp
-L Device:R R?
+L Device:R R59
 U 1 1 5F6A3EEE
 P 5000 2900
-F 0 "R?" H 5070 2946 50  0000 L CNN
+F 0 "R59" H 5070 2946 50  0000 L CNN
 F 1 "22k" H 5070 2855 50  0000 L CNN
 F 2 "" V 4930 2900 50  0001 C CNN
@@
 $EndComp
 $Comp
-L Device:R R?
+L Device:R R61
 U 1 1 5F6A3EF4
 P 5500 2900
-F 0 "R?" H 5570 2946 50  0000 L CNN
+F 0 "R61" H 5570 2946 50  0000 L CNN
 F 1 "22k" H 5570 2855 50  0000 L CNN
 F 2 "" V 5430 2900 50  0001 C CNN
@@
 $EndComp
 $Comp
-L Device:R R?
+L Device:R R63
 U 1 1 5F6A3EFA
 P 6000 2900
-F 0 "R?" H 6070 2946 50  0000 L CNN
+F 0 "R63" H 6070 2946 50  0000 L CNN
 F 1 "22k" H 6070 2855 50  0000 L CNN
 F 2 "" V 5930 2900 50  0001 C CNN
@@
 $EndComp
 $Comp
-L Device:R R?
+L Device:R R65
 U 1 1 5F6A3F00
 P 6500 2900
-F 0 "R?" H 6570 2946 50  0000 L CNN
+F 0 "R65" H 6570 2946 50  0000 L CNN
 F 1 "22k" H 6570 2855 50  0000 L CNN
 F 2 "" V 6430 2900 50  0001 C CNN
@@
 $EndComp
 $Comp
-L Device:R R?
+L Device:R R67
 U 1 1 5F6A3F06
 P 7000 2900
-F 0 "R?" H 7070 2946 50  0000 L CNN
+F 0 "R67" H 7070 2946 50  0000 L CNN
 F 1 "22k" H 7070 2855 50  0000 L CNN
 F 2 "" V 6930 2900 50  0001 C CNN
@@
 $EndComp
 $Comp
-L Device:R R?
+L Device:R R69
 U 1 1 5F6A3F0C
 P 7500 2900
-F 0 "R?" H 7570 2946 50  0000 L CNN
+F 0 "R69" H 7570 2946 50  0000 L CNN
 F 1 "22k" H 7570 2855 50  0000 L CNN
 F 2 "" V 7430 2900 50  0001 C CNN
@@
 P 5000 1800
 AR Path="/5F70A721/5F6A4A53" Ref="#PWR?"  Part="1"
-AR Path="/5F70B1A3/5F6A4A53" Ref="#PWR?"  Part="1"
-F 0 "#PWR?" H 5000 1550 50  0001 C CNN
+AR Path="/5F70B1A3/5F6A4A53" Ref="#PWR0158"  Part="1"
+F 0 "#PWR0158" H 5000 1550 50  0001 C CNN
 F 1 "GND" H 5005 1627 50  0000 C CNN
 F 2 "" H 5000 1800 50  0001 C CNN
@@
 P 5500 1800
 AR Path="/5F70A721/5F6A4F23" Ref="#PWR?"  Part="1"
-AR Path="/5F70B1A3/5F6A4F23" Ref="#PWR?"  Part="1"
-F 0 "#PWR?" H 5500 1550 50  0001 C CNN
+AR Path="/5F70B1A3/5F6A4F23" Ref="#PWR0159"  Part="1"
+F 0 "#PWR0159" H 5500 1550 50  0001 C CNN
 F 1 "GND" H 5505 1627 50  0000 C CNN
 F 2 "" H 5500 1800 50  0001 C CNN
@@
 P 6000 1800
 AR Path="/5F70A721/5F6A5197" Ref="#PWR?"  Part="1"
-AR Path="/5F70B1A3/5F6A5197" Ref="#PWR?"  Part="1"
-F 0 "#PWR?" H 6000 1550 50  0001 C CNN
+AR Path="/5F70B1A3/5F6A5197" Ref="#PWR0160"  Part="1"
+F 0 "#PWR0160" H 6000 1550 50  0001 C CNN
 F 1 "GND" H 6005 1627 50  0000 C CNN
 F 2 "" H 6000 1800 50  0001 C CNN
@@
 P 6500 1800
 AR Path="/5F70A721/5F6A5348" Ref="#PWR?"  Part="1"
-AR Path="/5F70B1A3/5F6A5348" Ref="#PWR?"  Part="1"
-F 0 "#PWR?" H 6500 1550 50  0001 C CNN
+AR Path="/5F70B1A3/5F6A5348" Ref="#PWR0161"  Part="1"
+F 0 "#PWR0161" H 6500 1550 50  0001 C CNN
 F 1 "GND" H 6505 1627 50  0000 C CNN
 F 2 "" H 6500 1800 50  0001 C CNN
@@
 P 7000 1800
 AR Path="/5F70A721/5F6A55E5" Ref="#PWR?"  Part="1"
-AR Path="/5F70B1A3/5F6A55E5" Ref="#PWR?"  Part="1"
-F 0 "#PWR?" H 7000 1550 50  0001 C CNN
+AR Path="/5F70B1A3/5F6A55E5" Ref="#PWR0162"  Part="1"
+F 0 "#PWR0162" H 7000 1550 50  0001 C CNN
 F 1 "GND" H 7005 1627 50  0000 C CNN
 F 2 "" H 7000 1800 50  0001 C CNN
@@
 P 7500 1800
 AR Path="/5F70A721/5F6A585F" Ref="#PWR?"  Part="1"
-AR Path="/5F70B1A3/5F6A585F" Ref="#PWR?"  Part="1"
-F 0 "#PWR?" H 7500 1550 50  0001 C CNN
+AR Path="/5F70B1A3/5F6A585F" Ref="#PWR0163"  Part="1"
+F 0 "#PWR0163" H 7500 1550 50  0001 C CNN
 F 1 "GND" H 7505 1627 50  0000 C CNN
 F 2 "" H 7500 1800 50  0001 C CNN
@@
 P 5000 3050
 AR Path="/5F70A721/5F6A59FF" Ref="#PWR?"  Part="1"
-AR Path="/5F70B1A3/5F6A59FF" Ref="#PWR?"  Part="1"
-F 0 "#PWR?" H 5000 2800 50  0001 C CNN
+AR Path="/5F70B1A3/5F6A59FF" Ref="#PWR0164"  Part="1"
+F 0 "#PWR0164" H 5000 2800 50  0001 C CNN
 F 1 "GND" H 5005 2877 50  0000 C CNN
 F 2 "" H 5000 3050 50  0001 C CNN
@@
 P 5500 3050
 AR Path="/5F70A721/5F6A5CE6" Ref="#PWR?"  Part="1"
-AR Path="/5F70B1A3/5F6A5CE6" Ref="#PWR?"  Part="1"
-F 0 "#PWR?" H 5500 2800 50  0001 C CNN
+AR Path="/5F70B1A3/5F6A5CE6" Ref="#PWR0165"  Part="1"
+F 0 "#PWR0165" H 5500 2800 50  0001 C CNN
 F 1 "GND" H 5505 2877 50  0000 C CNN
 F 2 "" H 5500 3050 50  0001 C CNN
@@
 P 6000 3050
 AR Path="/5F70A721/5F6A5EEC" Ref="#PWR?"  Part="1"
-AR Path="/5F70B1A3/5F6A5EEC" Ref="#PWR?"  Part="1"
-F 0 "#PWR?" H 6000 2800 50  0001 C CNN
+AR Path="/5F70B1A3/5F6A5EEC" Ref="#PWR0166"  Part="1"
+F 0 "#PWR0166" H 6000 2800 50  0001 C CNN
 F 1 "GND" H 6005 2877 50  0000 C CNN
 F 2 "" H 6000 3050 50  0001 C CNN
@@
 P 6500 3050
 AR Path="/5F70A721/5F6A6093" Ref="#PWR?"  Part="1"
-AR Path="/5F70B1A3/5F6A6093" Ref="#PWR?"  Part="1"
-F 0 "#PWR?" H 6500 2800 50  0001 C CNN
+AR Path="/5F70B1A3/5F6A6093" Ref="#PWR0167"  Part="1"
+F 0 "#PWR0167" H 6500 2800 50  0001 C CNN
 F 1 "GND" H 6505 2877 50  0000 C CNN
 F 2 "" H 6500 3050 50  0001 C CNN
@@
 P 7000 3050
 AR Path="/5F70A721/5F6A622C" Ref="#PWR?"  Part="1"
-AR Path="/5F70B1A3/5F6A622C" Ref="#PWR?"  Part="1"
-F 0 "#PWR?" H 7000 2800 50  0001 C CNN
+AR Path="/5F70B1A3/5F6A622C" Ref="#PWR0168"  Part="1"
+F 0 "#PWR0168" H 7000 2800 50  0001 C CNN
 F 1 "GND" H 7005 2877 50  0000 C CNN
 F 2 "" H 7000 3050 50  0001 C CNN
@@
 P 7500 3050
 AR Path="/5F70A721/5F6A6421" Ref="#PWR?"  Part="1"
-AR Path="/5F70B1A3/5F6A6421" Ref="#PWR?"  Part="1"
-F 0 "#PWR?" H 7500 2800 50  0001 C CNN
+AR Path="/5F70B1A3/5F6A6421" Ref="#PWR0169"  Part="1"
+F 0 "#PWR0169" H 7500 2800 50  0001 C CNN
 F 1 "GND" H 7505 2877 50  0000 C CNN
 F 2 "" H 7500 3050 50  0001 C CNN
