File: tempmux.sch (KiCad schematic (older format))
At the start: 23 parts, among them J7 Conn_02x07_Counter_Clockwise, U11 CD74HC4067SM

Commit message: Refactored some naming
Parts:
- renumbered J7 to J6
Changed lines of the file:
@@
 P 2000 3400
 AR Path="/5F70A721/5F6868D9" Ref="#PWR?"  Part="1"
-AR Path="/5F70B1A3/5F6868D9" Ref="#PWR077"  Part="1"
-F 0 "#PWR077" H 2000 3150 50  0001 C CNN
+AR Path="/5F70B1A3/5F6868D9" Ref="#PWR076"  Part="1"
+F 0 "#PWR076" H 2000 3150 50  0001 C CNN
 F 1 "GND" H 2005 3227 50  0000 C CNN
 F 2 "" H 2000 3400 50  0001 C CNN
@@
 P 2150 1200
 AR Path="/5F70A721/5F6868E6" Ref="#PWR?"  Part="1"
-AR Path="/5F70B1A3/5F6868E6" Ref="#PWR062"  Part="1"
-F 0 "#PWR062" H 2150 950 50  0001 C CNN
+AR Path="/5F70B1A3/5F6868E6" Ref="#PWR061"  Part="1"
+F 0 "#PWR061" H 2150 950 50  0001 C CNN
 F 1 "GND" H 2300 1150 50  0000 C CNN
 F 2 "" H 2150 1200 50  0001 C CNN
@@
 P 2000 950
 AR Path="/5F70A721/5F6868EC" Ref="#PWR?"  Part="1"
-AR Path="/5F70B1A3/5F6868EC" Ref="#PWR061"  Part="1"
-F 0 "#PWR061" H 2000 800 50  0001 C CNN
+AR Path="/5F70B1A3/5F6868EC" Ref="#PWR060"  Part="1"
+F 0 "#PWR060" H 2000 800 50  0001 C CNN
 F 1 "+5V" H 2015 1123 50  0000 C CNN
 F 2 "" H 2000 950 50  0001 C CNN
@@
 P 9900 1850
 AR Path="/5F70A721/5F68B135" Ref="J?"  Part="1"
-AR Path="/5F70B1A3/5F68B135" Ref="J7"  Part="1"
-F 0 "J7" H 9950 2300 50  0000 C CNN
+AR Path="/5F70B1A3/5F68B135" Ref="J6"  Part="1"
+F 0 "J6" H 9950 2300 50  0000 C CNN
 F 1 "Conn_02x07_Counter_Clockwise" H 9950 1450 50  0000 C CNN
 F 2 "Connector_PinHeader_2.54mm:PinHeader_2x07_P2.54mm_Vertical" H 9900 1850 50  0001 C CNN
@@
 P 9650 1550
 AR Path="/5F70A721/5F68DF75" Ref="#PWR?"  Part="1"
-AR Path="/5F70B1A3/5F68DF75" Ref="#PWR063"  Part="1"
-F 0 "#PWR063" H 9650 1400 50  0001 C CNN
+AR Path="/5F70B1A3/5F68DF75" Ref="#PWR062"  Part="1"
+F 0 "#PWR062" H 9650 1400 50  0001 C CNN
 F 1 "+5V" H 9665 1723 50  0000 C CNN
 F 2 "" H 9650 1550 50  0001 C CNN
@@
 P 10250 1550
 AR Path="/5F70A721/5F68E7C7" Ref="#PWR?"  Part="1"
-AR Path="/5F70B1A3/5F68E7C7" Ref="#PWR064"  Part="1"
-F 0 "#PWR064" H 10250 1400 50  0001 C CNN
+AR Path="/5F70B1A3/5F68E7C7" Ref="#PWR063"  Part="1"
+F 0 "#PWR063" H 10250 1400 50  0001 C CNN
 F 1 "+5V" H 10265 1723 50  0000 C CNN
 F 2 "" H 10250 1550 50  0001 C CNN
@@
 P 5000 1800
 AR Path="/5F70A721/5F6A4A53" Ref="#PWR?"  Part="1"
-AR Path="/5F70B1A3/5F6A4A53" Ref="#PWR065"  Part="1"
-F 0 "#PWR065" H 5000 1550 50  0001 C CNN
+AR Path="/5F70B1A3/5F6A4A53" Ref="#PWR064"  Part="1"
+F 0 "#PWR064" H 5000 1550 50  0001 C CNN
 F 1 "GND" H 5005 1627 50  0000 C CNN
 F 2 "" H 5000 1800 50  0001 C CNN
@@
 P 5500 1800
 AR Path="/5F70A721/5F6A4F23" Ref="#PWR?"  Part="1"
-AR Path="/5F70B1A3/5F6A4F23" Ref="#PWR066"  Part="1"
-F 0 "#PWR066" H 5500 1550 50  0001 C CNN
+AR Path="/5F70B1A3/5F6A4F23" Ref="#PWR065"  Part="1"
+F 0 "#PWR065" H 5500 1550 50  0001 C CNN
 F 1 "GND" H 5505 1627 50  0000 C CNN
 F 2 "" H 5500 1800 50  0001 C CNN
@@
 P 6000 1800
 AR Path="/5F70A721/5F6A5197" Ref="#PWR?"  Part="1"
-AR Path="/5F70B1A3/5F6A5197" Ref="#PWR067"  Part="1"
-F 0 "#PWR067" H 6000 1550 50  0001 C CNN
+AR Path="/5F70B1A3/5F6A5197" Ref="#PWR066"  Part="1"
+F 0 "#PWR066" H 6000 1550 50  0001 C CNN
 F 1 "GND" H 6005 1627 50  0000 C CNN
 F 2 "" H 6000 1800 50  0001 C CNN
@@
 P 6500 1800
 AR Path="/5F70A721/5F6A5348" Ref="#PWR?"  Part="1"
-AR Path="/5F70B1A3/5F6A5348" Ref="#PWR068"  Part="1"
-F 0 "#PWR068" H 6500 1550 50  0001 C CNN
+AR Path="/5F70B1A3/5F6A5348" Ref="#PWR067"  Part="1"
+F 0 "#PWR067" H 6500 1550 50  0001 C CNN
 F 1 "GND" H 6505 1627 50  0000 C CNN
 F 2 "" H 6500 1800 50  0001 C CNN
@@
 P 7000 1800
 AR Path="/5F70A721/5F6A55E5" Ref="#PWR?"  Part="1"
-AR Path="/5F70B1A3/5F6A55E5" Ref="#PWR069"  Part="1"
-F 0 "#PWR069" H 7000 1550 50  0001 C CNN
+AR Path="/5F70B1A3/5F6A55E5" Ref="#PWR068"  Part="1"
+F 0 "#PWR068" H 7000 1550 50  0001 C CNN
 F 1 "GND" H 7005 1627 50  0000 C CNN
 F 2 "" H 7000 1800 50  0001 C CNN
@@
 P 7500 1800
 AR Path="/5F70A721/5F6A585F" Ref="#PWR?"  Part="1"
-AR Path="/5F70B1A3/5F6A585F" Ref="#PWR070"  Part="1"
-F 0 "#PWR070" H 7500 1550 50  0001 C CNN
+AR Path="/5F70B1A3/5F6A585F" Ref="#PWR069"  Part="1"
+F 0 "#PWR069" H 7500 1550 50  0001 C CNN
 F 1 "GND" H 7505 1627 50  0000 C CNN
 F 2 "" H 7500 1800 50  0001 C CNN
@@
 P 5000 3050
 AR Path="/5F70A721/5F6A59FF" Ref="#PWR?"  Part="1"
-AR Path="/5F70B1A3/5F6A59FF" Ref="#PWR071"  Part="1"
-F 0 "#PWR071" H 5000 2800 50  0001 C CNN
+AR Path="/5F70B1A3/5F6A59FF" Ref="#PWR070"  Part="1"
+F 0 "#PWR070" H 5000 2800 50  0001 C CNN
 F 1 "GND" H 5005 2877 50  0000 C CNN
 F 2 "" H 5000 3050 50  0001 C CNN
@@
 P 5500 3050
 AR Path="/5F70A721/5F6A5CE6" Ref="#PWR?"  Part="1"
-AR Path="/5F70B1A3/5F6A5CE6" Ref="#PWR072"  Part="1"
-F 0 "#PWR072" H 5500 2800 50  0001 C CNN
+AR Path="/5F70B1A3/5F6A5CE6" Ref="#PWR071"  Part="1"
+F 0 "#PWR071" H 5500 2800 50  0001 C CNN
 F 1 "GND" H 5505 2877 50  0000 C CNN
 F 2 "" H 5500 3050 50  0001 C CNN
@@
 P 6000 3050
 AR Path="/5F70A721/5F6A5EEC" Ref="#PWR?"  Part="1"
-AR Path="/5F70B1A3/5F6A5EEC" Ref="#PWR073"  Part="1"
-F 0 "#PWR073" H 6000 2800 50  0001 C CNN
+AR Path="/5F70B1A3/5F6A5EEC" Ref="#PWR072"  Part="1"
+F 0 "#PWR072" H 6000 2800 50  0001 C CNN
 F 1 "GND" H 6005 2877 50  0000 C CNN
 F 2 "" H 6000 3050 50  0001 C CNN
@@
 P 6500 3050
 AR Path="/5F70A721/5F6A6093" Ref="#PWR?"  Part="1"
-AR Path="/5F70B1A3/5F6A6093" Ref="#PWR074"  Part="1"
-F 0 "#PWR074" H 6500 2800 50  0001 C CNN
+AR Path="/5F70B1A3/5F6A6093" Ref="#PWR073"  Part="1"
+F 0 "#PWR073" H 6500 2800 50  0001 C CNN
 F 1 "GND" H 6505 2877 50  0000 C CNN
 F 2 "" H 6500 3050 50  0001 C CNN
@@
 P 7000 3050
 AR Path="/5F70A721/5F6A622C" Ref="#PWR?"  Part="1"
-AR Path="/5F70B1A3/5F6A622C" Ref="#PWR075"  Part="1"
-F 0 "#PWR075" H 7000 2800 50  0001 C CNN
+AR Path="/5F70B1A3/5F6A622C" Ref="#PWR074"  Part="1"
+F 0 "#PWR074" H 7000 2800 50  0001 C CNN
 F 1 "GND" H 7005 2877 50  0000 C CNN
 F 2 "" H 7000 3050 50  0001 C CNN
@@
 P 7500 3050
 AR Path="/5F70A721/5F6A6421" Ref="#PWR?"  Part="1"
-AR Path="/5F70B1A3/5F6A6421" Ref="#PWR076"  Part="1"
-F 0 "#PWR076" H 7500 2800 50  0001 C CNN
+AR Path="/5F70B1A3/5F6A6421" Ref="#PWR075"  Part="1"
+F 0 "#PWR075" H 7500 2800 50  0001 C CNN
 F 1 "GND" H 7505 2877 50  0000 C CNN
 F 2 "" H 7500 3050 50  0001 C CNN
@@
 P 5000 4450
 AR Path="/5F70A721/5F26879D" Ref="#PWR?"  Part="1"
-AR Path="/5F70B1A3/5F26879D" Ref="#PWR082"  Part="1"
-F 0 "#PWR082" H 5000 4200 50  0001 C CNN
+AR Path="/5F70B1A3/5F26879D" Ref="#PWR081"  Part="1"
+F 0 "#PWR081" H 5000 4200 50  0001 C CNN
 F 1 "GND" H 5005 4277 50  0000 C CNN
 F 2 "" H 5000 4450 50  0001 C CNN
@@
 P 5000 3650
 AR Path="/5F70A721/5F269BD4" Ref="#PWR?"  Part="1"
-AR Path="/5F70B1A3/5F269BD4" Ref="#PWR078"  Part="1"
-F 0 "#PWR078" H 5000 3500 50  0001 C CNN
+AR Path="/5F70B1A3/5F269BD4" Ref="#PWR077"  Part="1"
+F 0 "#PWR077" H 5000 3500 50  0001 C CNN
 F 1 "+5V" H 5015 3823 50  0000 C CNN
 F 2 "" H 5000 3650 50  0001 C CNN
@@
 P 6000 4450
 AR Path="/5F70A721/5F26E1A4" Ref="#PWR?"  Part="1"
-AR Path="/5F70B1A3/5F26E1A4" Ref="#PWR083"  Part="1"
-F 0 "#PWR083" H 6000 4200 50  0001 C CNN
+AR Path="/5F70B1A3/5F26E1A4" Ref="#PWR082"  Part="1"
+F 0 "#PWR082" H 6000 4200 50  0001 C CNN
 F 1 "GND" H 6005 4277 50  0000 C CNN
 F 2 "" H 6000 4450 50  0001 C CNN
@@
 P 6000 3650
 AR Path="/5F70A721/5F26E1AB" Ref="#PWR?"  Part="1"
-AR Path="/5F70B1A3/5F26E1AB" Ref="#PWR079"  Part="1"
-F 0 "#PWR079" H 6000 3500 50  0001 C CNN
+AR Path="/5F70B1A3/5F26E1AB" Ref="#PWR078"  Part="1"
+F 0 "#PWR078" H 6000 3500 50  0001 C CNN
 F 1 "+5V" H 6015 3823 50  0000 C CNN
 F 2 "" H 6000 3650 50  0001 C CNN
@@
 P 7000 4450
 AR Path="/5F70A721/5F2705CC" Ref="#PWR?"  Part="1"
-AR Path="/5F70B1A3/5F2705CC" Ref="#PWR084"  Part="1"
-F 0 "#PWR084" H 7000 4200 50  0001 C CNN
+AR Path="/5F70B1A3/5F2705CC" Ref="#PWR083"  Part="1"
+F 0 "#PWR083" H 7000 4200 50  0001 C CNN
 F 1 "GND" H 7005 4277 50  0000 C CNN
 F 2 "" H 7000 4450 50  0001 C CNN
@@
 P 7000 3650
 AR Path="/5F70A721/5F2705D3" Ref="#PWR?"  Part="1"
-AR Path="/5F70B1A3/5F2705D3" Ref="#PWR080"  Part="1"
-F 0 "#PWR080" H 7000 3500 50  0001 C CNN
+AR Path="/5F70B1A3/5F2705D3" Ref="#PWR079"  Part="1"
+F 0 "#PWR079" H 7000 3500 50  0001 C CNN
 F 1 "+5V" H 7015 3823 50  0000 C CNN
 F 2 "" H 7000 3650 50  0001 C CNN
@@
 P 8000 4450
 AR Path="/5F70A721/5F272D66" Ref="#PWR?"  Part="1"
-AR Path="/5F70B1A3/5F272D66" Ref="#PWR085"  Part="1"
-F 0 "#PWR085" H 8000 4200 50  0001 C CNN
+AR Path="/5F70B1A3/5F272D66" Ref="#PWR084"  Part="1"
+F 0 "#PWR084" H 8000 4200 50  0001 C CNN
 F 1 "GND" H 8005 4277 50  0000 C CNN
 F 2 "" H 8000 4450 50  0001 C CNN
@@
 P 8000 3650
 AR Path="/5F70A721/5F272D6D" Ref="#PWR?"  Part="1"
-AR Path="/5F70B1A3/5F272D6D" Ref="#PWR081"  Part="1"
-F 0 "#PWR081" H 8000 3500 50  0001 C CNN
+AR Path="/5F70B1A3/5F272D6D" Ref="#PWR080"  Part="1"
+F 0 "#PWR080" H 8000 3500 50  0001 C CNN
 F 1 "+5V" H 8015 3823 50  0000 C CNN
 F 2 "" H 8000 3650 50  0001 C CNN

Commit message: Added new 14 pin connector footprint
Parts:
- J6: footprint Connector_PinHeader_2.54mm:PinHeader_2x07_P2.54mm_Vertical -> uBMS-2:CNC-Tech_3020-14-0300-00
Changed lines of the file:
@@
 F 0 "J6" H 9950 2300 50  0000 C CNN
 F 1 "Conn_02x07_Counter_Clockwise" H 9950 1450 50  0000 C CNN
-F 2 "Connector_PinHeader_2.54mm:PinHeader_2x07_P2.54mm_Vertical" H 9900 1850 50  0001 C CNN
+F 2 "uBMS-2:CNC-Tech_3020-14-0300-00" H 9900 1850 50  0001 C CNN
 F 3 "~" H 9900 1850 50  0001 C CNN
 	1    9900 1850

Commit message: Using Molex Milli Grid Connector for 14 pin
Parts:
- J6: footprint uBMS-2:CNC-Tech_3020-14-0300-00 -> uBMS-2:Molex_Milli_Grid_0878325623
Changed lines of the file:
@@
 F 0 "J6" H 9950 2300 50  0000 C CNN
 F 1 "Conn_02x07_Counter_Clockwise" H 9950 1450 50  0000 C CNN
-F 2 "uBMS-2:CNC-Tech_3020-14-0300-00" H 9900 1850 50  0001 C CNN
+F 2 "uBMS-2:Molex_Milli_Grid_0878325623" H 9900 1850 50  0001 C CNN
 F 3 "~" H 9900 1850 50  0001 C CNN
 	1    9900 1850

Commit message: routed and filled a bunch of stuff, so much more to do
Parts:
- removed J6: Conn_02x07_Counter_Clockwise, uBMS-2:Molex_Milli_Grid_0878325623, symbol Connector_Generic:Conn_02x07_Counter_Clockwise
- added J6: Conn_02x07_Odd_Even, uBMS-2:Molex_Milli_Grid_0878325623_TopBottom, symbol Connector_Generic:Conn_02x07_Odd_Even
Connections:
- net +5V: now also J6.13 (Pin_13), J6.14 (Pin_14)
- net CellTemp_1: now also J6.1 (Pin_1)
- net CellTemp_10: now also J6.10 (Pin_10)
- net CellTemp_11: now also J6.11 (Pin_11)
- net CellTemp_12: now also J6.12 (Pin_12)
- net CellTemp_2: now also J6.2 (Pin_2)
- net CellTemp_3: now also J6.3 (Pin_3)
- net CellTemp_4: now also J6.4 (Pin_4)
- net CellTemp_5: now also J6.5 (Pin_5)
- net CellTemp_6: now also J6.6 (Pin_6)
- net CellTemp_7: now also J6.7 (Pin_7)
- net CellTemp_8: now also J6.8 (Pin_8)
- net CellTemp_9: now also J6.9 (Pin_9)
Changed lines of the file:
@@
 	1450 2800 1500 2800
-$Comp
-L Connector_Generic:Conn_02x07_Counter_Clockwise J?
-U 1 1 5F68B135
-P 9900 1850
-AR Path="/5F70A721/5F68B135" Ref="J?"  Part="1"
-AR Path="/5F70B1A3/5F68B135" Ref="J6"  Part="1"
-F 0 "J6" H 9950 2300 50  0000 C CNN
-F 1 "Conn_02x07_Counter_Clockwise" H 9950 1450 50  0000 C CNN
-F 2 "uBMS-2:Molex_Milli_Grid_0878325623" H 9900 1850 50  0001 C CNN
-F 3 "~" H 9900 1850 50  0001 C CNN
-	1    9900 1850
-	1    0    0    -1
-$EndComp
 $Comp
 L power:+5V #PWR?
 U 1 1 5F68DF75
-P 9650 1550
+P 9000 2150
 AR Path="/5F70A721/5F68DF75" Ref="#PWR?"  Part="1"
 AR Path="/5F70B1A3/5F68DF75" Ref="#PWR062"  Part="1"
-F 0 "#PWR062" H 9650 1400 50  0001 C CNN
-F 1 "+5V" H 9665 1723 50  0000 C CNN
-F 2 "" H 9650 1550 50  0001 C CNN
-F 3 "" H 9650 1550 50  0001 C CNN
-	1    9650 1550
+F 0 "#PWR062" H 9000 2000 50  0001 C CNN
+F 1 "+5V" H 9015 2323 50  0000 C CNN
+F 2 "" H 9000 2150 50  0001 C CNN
+F 3 "" H 9000 2150 50  0001 C CNN
+	1    9000 2150
 	1    0    0    -1
 $EndComp
@@
 L power:+5V #PWR?
 U 1 1 5F68E7C7
-P 10250 1550
+P 10850 2150
 AR Path="/5F70A721/5F68E7C7" Ref="#PWR?"  Part="1"
 AR Path="/5F70B1A3/5F68E7C7" Ref="#PWR063"  Part="1"
-F 0 "#PWR063" H 10250 1400 50  0001 C CNN
-F 1 "+5V" H 10265 1723 50  0000 C CNN
-F 2 "" H 10250 1550 50  0001 C CNN
-F 3 "" H 10250 1550 50  0001 C CNN
-	1    10250 1550
-	1    0    0    -1
-$EndComp
-Wire Wire Line
-	10250 1550 10200 1550
-Wire Wire Line
-	9700 1550 9650 1550
+F 0 "#PWR063" H 10850 2000 50  0001 C CNN
+F 1 "+5V" H 10865 2323 50  0000 C CNN
+F 2 "" H 10850 2150 50  0001 C CNN
+F 3 "" H 10850 2150 50  0001 C CNN
+	1    10850 2150
+	1    0    0    -1
+$EndComp
+Text Label 9600 1550 2    50   ~ 0
+CellTemp_1
+Text Label 10300 1550 0    50   ~ 0
+CellTemp_2
 Text Label 9600 1650 2    50   ~ 0
-CellTemp_1
+CellTemp_3
+Text Label 10300 1650 0    50   ~ 0
+CellTemp_4
 Text Label 9600 1750 2    50   ~ 0
-CellTemp_2
+CellTemp_5
+Text Label 10300 1750 0    50   ~ 0
+CellTemp_6
 Text Label 9600 1850 2    50   ~ 0
-CellTemp_3
+CellTemp_7
+Text Label 10300 1850 0    50   ~ 0
+CellTemp_8
 Text Label 9600 1950 2    50   ~ 0
-CellTemp_4
+CellTemp_9
+Text Label 10300 1950 0    50   ~ 0
+CellTemp_10
 Text Label 9600 2050 2    50   ~ 0
-CellTemp_5
-Text Label 9600 2150 2    50   ~ 0
-CellTemp_6
-Text Label 10300 2150 0    50   ~ 0
-CellTemp_7
+CellTemp_11
 Text Label 10300 2050 0    50   ~ 0
-CellTemp_8
-Text Label 10300 1950 0    50   ~ 0
-CellTemp_9
-Text Label 10300 1850 0    50   ~ 0
-CellTemp_10
-Text Label 10300 1750 0    50   ~ 0
-CellTemp_11
-Text Label 10300 1650 0    50   ~ 0
 CellTemp_12
 Wire Wire Line
@@
 Wire Wire Line
 	9600 2050 9700 2050
-Wire Wire Line
-	9600 2150 9700 2150
-Wire Wire Line
-	10200 2150 10300 2150
 Wire Wire Line
 	10200 2050 10300 2050
@@
 Wire Wire Line
 	2500 3000 2600 3000
+$Comp
+L Connector_Generic:Conn_02x07_Odd_Even J6
+U 1 1 5F36EBDC
+P 9900 1850
+F 0 "J6" H 9950 2367 50  0000 C CNN
+F 1 "Conn_02x07_Odd_Even" H 9950 2276 50  0000 C CNN
+F 2 "uBMS-2:Molex_Milli_Grid_0878325623_TopBottom" H 9900 1850 50  0001 C CNN
+F 3 "~" H 9900 1850 50  0001 C CNN
+	1    9900 1850
+	1    0    0    -1
+$EndComp
+Wire Wire Line
+	10200 1550 10300 1550
+Wire Wire Line
+	9600 1550 9700 1550
+Wire Wire Line
+	9000 2150 9700 2150
+Wire Wire Line
+	10200 2150 10850 2150
 $EndSCHEMATC
