File: tempmux.sch (KiCad schematic (older format))
At the start: 23 parts, among them J6 Conn_02x07_Odd_Even, U11 CD74HC4067SM

Commit message: Updated all the caps (I think) mostly changed to 0805
- Added 0603 footprints to new resistors which is slightly different from the old 0603 resistors for some reason???
- Annotated the schematic
- Still need to do the inductor oof
Parts:
- C14: footprint Capacitor_SMD:C_1206_3216Metric -> Capacitor_SMD:C_0805_2012Metric; Comment (none) -> 0.1µF -20%, +80% 16V Ceramic Capacitor Y5V 0805 (2012 Metri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; Digikey Number (none) -> 399-9159-2-ND; Part Number (none) -> C0805C104Z4VACTU; Price ($) (none) -> 0.11
Changed lines of the file:
@@
-$EndComp
-$Comp
-L Device:C_Small C?
-U 1 1 5F6868E0
-P 2150 1100
-AR Path="/5F70A721/5F6868E0" Ref="C?"  Part="1"
-AR Path="/5F70B1A3/5F6868E0" Ref="C14"  Part="1"
-F 0 "C14" H 2242 1146 50  0000 L CNN
-F 1 "0.1uF" H 2242 1055 50  0000 L CNN
-F 2 "Capacitor_SMD:C_1206_3216Metric" H 2150 1100 50  0001 C CNN
-F 3 "~" H 2150 1100 50  0001 C CNN
-	1    2150 1100
-	1    0    0    -1
 $EndComp
 $Comp
@@
 Wire Wire Line
 	10200 2150 10850 2150
+$Comp
+L Device:C_Small C?
+U 1 1 5FD78D93
+P 2150 1100
+AR Path="/5FD78D93" Ref="C?"  Part="1"
+AR Path="/5F70B1A3/5FD78D93" Ref="C14"  Part="1"
+F 0 "C14" H 2242 1146 50  0000 L CNN
+F 1 "0.1uF" H 2242 1055 50  0000 L CNN
+F 2 "Capacitor_SMD:C_0805_2012Metric" H 2150 1100 50  0001 C CNN
+F 3 "https://content.kemet.com/datasheets/KEM_C1005_Y5V_SMD.pdf" H 2150 1100 50  0001 C CNN
+F 4 "C0805C104Z4VACTU" H 2150 1100 50  0001 C CNN "Part Number"
+F 5 "399-9159-2-ND" H 2150 1100 50  0001 C CNN "Digikey Number"
+F 6 "0.11" H 2150 1100 50  0001 C CNN "Price ($)"
+F 7 "0.1µF -20%, +80% 16V Ceramic Capacitor Y5V 0805 (2012 Metric)" H 2150 1100 50  0001 C CNN "Comment"
+	1    2150 1100
+	1    0    0    -1
+$EndComp
 $EndSCHEMATC

Commit message: Reset 0604 resistors to smaller (older?) footprint size
Parts:
- R60, R61, R62, R63, R64, R65, R66, R67, R68, R69, R70, R71, R72, R73, R74, R75: footprint Resistor_SMD:R_0603_1608Metric_Pad1.05x0.95mm_HandSolder -> Resistor_SMD:R_0603_1608Metric_Pad0.98x0.95mm_HandSolder
Changed lines of the file:
@@
 F 0 "R60" H 5070 1696 50  0000 L CNN
 F 1 "22k" H 5070 1605 50  0000 L CNN
-F 2 "Resistor_SMD:R_0603_1608Metric_Pad1.05x0.95mm_HandSolder" V 4930 1650 50  0001 C CNN
+F 2 "Resistor_SMD:R_0603_1608Metric_Pad0.98x0.95mm_HandSolder" V 4930 1650 50  0001 C CNN
 F 3 "~" H 5000 1650 50  0001 C CNN
 	1    5000 1650
@@
 F 0 "R61" H 5570 1696 50  0000 L CNN
 F 1 "22k" H 5570 1605 50  0000 L CNN
-F 2 "Resistor_SMD:R_0603_1608Metric_Pad1.05x0.95mm_HandSolder" V 5430 1650 50  0001 C CNN
+F 2 "Resistor_SMD:R_0603_1608Metric_Pad0.98x0.95mm_HandSolder" V 5430 1650 50  0001 C CNN
 F 3 "~" H 5500 1650 50  0001 C CNN
 	1    5500 1650
@@
 F 0 "R62" H 6070 1696 50  0000 L CNN
 F 1 "22k" H 6070 1605 50  0000 L CNN
-F 2 "Resistor_SMD:R_0603_1608Metric_Pad1.05x0.95mm_HandSolder" V 5930 1650 50  0001 C CNN
+F 2 "Resistor_SMD:R_0603_1608Metric_Pad0.98x0.95mm_HandSolder" V 5930 1650 50  0001 C CNN
 F 3 "~" H 6000 1650 50  0001 C CNN
 	1    6000 1650
@@
 F 0 "R63" H 6570 1696 50  0000 L CNN
 F 1 "22k" H 6570 1605 50  0000 L CNN
-F 2 "Resistor_SMD:R_0603_1608Metric_Pad1.05x0.95mm_HandSolder" V 6430 1650 50  0001 C CNN
+F 2 "Resistor_SMD:R_0603_1608Metric_Pad0.98x0.95mm_HandSolder" V 6430 1650 50  0001 C CNN
 F 3 "~" H 6500 1650 50  0001 C CNN
 	1    6500 1650
@@
 F 0 "R64" H 7070 1696 50  0000 L CNN
 F 1 "22k" H 7070 1605 50  0000 L CNN
-F 2 "Resistor_SMD:R_0603_1608Metric_Pad1.05x0.95mm_HandSolder" V 6930 1650 50  0001 C CNN
+F 2 "Resistor_SMD:R_0603_1608Metric_Pad0.98x0.95mm_HandSolder" V 6930 1650 50  0001 C CNN
 F 3 "~" H 7000 1650 50  0001 C CNN
 	1    7000 1650
@@
 F 0 "R65" H 7570 1696 50  0000 L CNN
 F 1 "22k" H 7570 1605 50  0000 L CNN
-F 2 "Resistor_SMD:R_0603_1608Metric_Pad1.05x0.95mm_HandSolder" V 7430 1650 50  0001 C CNN
+F 2 "Resistor_SMD:R_0603_1608Metric_Pad0.98x0.95mm_HandSolder" V 7430 1650 50  0001 C CNN
 F 3 "~" H 7500 1650 50  0001 C CNN
 	1    7500 1650
@@
 F 0 "R66" H 5070 2946 50  0000 L CNN
 F 1 "22k" H 5070 2855 50  0000 L CNN
-F 2 "Resistor_SMD:R_0603_1608Metric_Pad1.05x0.95mm_HandSolder" V 4930 2900 50  0001 C CNN
+F 2 "Resistor_SMD:R_0603_1608Metric_Pad0.98x0.95mm_HandSolder" V 4930 2900 50  0001 C CNN
 F 3 "~" H 5000 2900 50  0001 C CNN
 	1    5000 2900
@@
 F 0 "R67" H 5570 2946 50  0000 L CNN
 F 1 "22k" H 5570 2855 50  0000 L CNN
-F 2 "Resistor_SMD:R_0603_1608Metric_Pad1.05x0.95mm_HandSolder" V 5430 2900 50  0001 C CNN
+F 2 "Resistor_SMD:R_0603_1608Metric_Pad0.98x0.95mm_HandSolder" V 5430 2900 50  0001 C CNN
 F 3 "~" H 5500 2900 50  0001 C CNN
 	1    5500 2900
@@
 F 0 "R68" H 6070 2946 50  0000 L CNN
 F 1 "22k" H 6070 2855 50  0000 L CNN
-F 2 "Resistor_SMD:R_0603_1608Metric_Pad1.05x0.95mm_HandSolder" V 5930 2900 50  0001 C CNN
+F 2 "Resistor_SMD:R_0603_1608Metric_Pad0.98x0.95mm_HandSolder" V 5930 2900 50  0001 C CNN
 F 3 "~" H 6000 2900 50  0001 C CNN
 	1    6000 2900
@@
 F 0 "R69" H 6570 2946 50  0000 L CNN
 F 1 "22k" H 6570 2855 50  0000 L CNN
-F 2 "Resistor_SMD:R_0603_1608Metric_Pad1.05x0.95mm_HandSolder" V 6430 2900 50  0001 C CNN
+F 2 "Resistor_SMD:R_0603_1608Metric_Pad0.98x0.95mm_HandSolder" V 6430 2900 50  0001 C CNN
 F 3 "~" H 6500 2900 50  0001 C CNN
 	1    6500 2900
@@
 F 0 "R70" H 7070 2946 50  0000 L CNN
 F 1 "22k" H 7070 2855 50  0000 L CNN
-F 2 "Resistor_SMD:R_0603_1608Metric_Pad1.05x0.95mm_HandSolder" V 6930 2900 50  0001 C CNN
+F 2 "Resistor_SMD:R_0603_1608Metric_Pad0.98x0.95mm_HandSolder" V 6930 2900 50  0001 C CNN
 F 3 "~" H 7000 2900 50  0001 C CNN
 	1    7000 2900
@@
 F 0 "R71" H 7570 2946 50  0000 L CNN
 F 1 "22k" H 7570 2855 50  0000 L CNN
-F 2 "Resistor_SMD:R_0603_1608Metric_Pad1.05x0.95mm_HandSolder" V 7430 2900 50  0001 C CNN
+F 2 "Resistor_SMD:R_0603_1608Metric_Pad0.98x0.95mm_HandSolder" V 7430 2900 50  0001 C CNN
 F 3 "~" H 7500 2900 50  0001 C CNN
 	1    7500 2900
@@
 F 0 "R72" H 5070 4296 50  0000 L CNN
 F 1 "4.7k" H 5070 4205 50  0000 L CNN
-F 2 "Resistor_SMD:R_0603_1608Metric_Pad1.05x0.95mm_HandSolder" V 4930 4250 50  0001 C CNN
+F 2 "Resistor_SMD:R_0603_1608Metric_Pad0.98x0.95mm_HandSolder" V 4930 4250 50  0001 C CNN
 F 3 "~" H 5000 4250 50  0001 C CNN
 	1    5000 4250
@@
 F 0 "R73" H 6070 4296 50  0000 L CNN
 F 1 "4.7k" H 6070 4205 50  0000 L CNN
-F 2 "Resistor_SMD:R_0603_1608Metric_Pad1.05x0.95mm_HandSolder" V 5930 4250 50  0001 C CNN
+F 2 "Resistor_SMD:R_0603_1608Metric_Pad0.98x0.95mm_HandSolder" V 5930 4250 50  0001 C CNN
 F 3 "~" H 6000 4250 50  0001 C CNN
 	1    6000 4250
@@
 F 0 "R74" H 7070 4296 50  0000 L CNN
 F 1 "4.7k" H 7070 4205 50  0000 L CNN
-F 2 "Resistor_SMD:R_0603_1608Metric_Pad1.05x0.95mm_HandSolder" V 6930 4250 50  0001 C CNN
+F 2 "Resistor_SMD:R_0603_1608Metric_Pad0.98x0.95mm_HandSolder" V 6930 4250 50  0001 C CNN
 F 3 "~" H 7000 4250 50  0001 C CNN
 	1    7000 4250
@@
 F 0 "R75" H 8070 4296 50  0000 L CNN
 F 1 "4.7k" H 8070 4205 50  0000 L CNN
-F 2 "Resistor_SMD:R_0603_1608Metric_Pad1.05x0.95mm_HandSolder" V 7930 4250 50  0001 C CNN
+F 2 "Resistor_SMD:R_0603_1608Metric_Pad0.98x0.95mm_HandSolder" V 7930 4250 50  0001 C CNN
 F 3 "~" H 8000 4250 50  0001 C CNN
 	1    8000 4250

Commit message: Finish PCB Layout Preliminary
- Moved around temp connections to the analogue mux to help aid layout
- Moved around voltage sense connections too
- Moved around LED status shift reg
- " and the 7 seg shift reg
- Added filled copper layers
- Removed external ADC Input
Connections:
- net Balance_Temp: now also U11.8 (I1); no longer U11.18 (I13)
- net CellTemp_1: now also U11.23 (I8); no longer U11.9 (I0)
- net CellTemp_10: now also U11.6 (I3); no longer U11.22 (I9)
- net CellTemp_11: now also U11.18 (I13); no longer U11.21 (I10)
- net CellTemp_12: now also U11.7 (I2); no longer U11.20 (I11)
- net CellTemp_2: now also U11.2 (I7); no longer U11.8 (I1)
- net CellTemp_3: now also U11.22 (I9); no longer U11.7 (I2)
- net CellTemp_4: now also U11.3 (I6); no longer U11.6 (I3)
- net CellTemp_5: now also U11.21 (I10); no longer U11.5 (I4)
- net CellTemp_7: now also U11.20 (I11); no longer U11.3 (I6)
- net CellTemp_8: now also U11.5 (I4); no longer U11.2 (I7)
- net CellTemp_9: now also U11.19 (I12); no longer U11.23 (I8)
- net Mosfet_Temp: now also U11.9 (I0); no longer U11.19 (I12)
Changed lines of the file:
@@
 Wire Wire Line
 	7500 2700 7500 2750
-Text Label 2600 1500 0    50   ~ 0
+Text Label 2600 2300 0    50   ~ 0
 CellTemp_1
-Text Label 2600 1600 0    50   ~ 0
+Text Label 2600 2200 0    50   ~ 0
 CellTemp_2
-Text Label 2600 1700 0    50   ~ 0
+Text Label 2600 2400 0    50   ~ 0
 CellTemp_3
-Text Label 2600 1800 0    50   ~ 0
+Text Label 2600 2100 0    50   ~ 0
 CellTemp_4
-Text Label 2600 1900 0    50   ~ 0
+Text Label 2600 2500 0    50   ~ 0
 CellTemp_5
 Text Label 2600 2000 0    50   ~ 0
 CellTemp_6
-Text Label 2600 2100 0    50   ~ 0
+Text Label 2600 2600 0    50   ~ 0
 CellTemp_7
-Text Label 2600 2200 0    50   ~ 0
+Text Label 2600 1900 0    50   ~ 0
 CellTemp_8
-Text Label 2600 2300 0    50   ~ 0
+Text Label 2600 2700 0    50   ~ 0
 CellTemp_9
-Text Label 2600 2400 0    50   ~ 0
+Text Label 2600 1800 0    50   ~ 0
 CellTemp_10
-Text Label 2600 2500 0    50   ~ 0
+Text Label 2600 2800 0    50   ~ 0
 CellTemp_11
-Text Label 2600 2600 0    50   ~ 0
+Text Label 2600 1700 0    50   ~ 0
 CellTemp_12
 Wire Wire Line
@@
 Wire Wire Line
 	8000 3650 8000 3700
-Text Label 2600 2700 0    50   ~ 0
+Text Label 2600 1500 0    50   ~ 0
 Mosfet_Temp
 Wire Wire Line
@@
 Text Label 4850 4050 2    50   ~ 0
 Mosfet_Temp
-Text Label 2600 2800 0    50   ~ 0
+Text Label 2600 1600 0    50   ~ 0
 Balance_Temp
 Text Label 2600 2900 0    50   ~ 0

Commit message: Updated some properties and generated BOM with KiBOM
Parts:
- J6: Comment (none) -> Connector Header Surface Mount 14 position 0.079\" (2.00mm); Digikey Number (none) -> WM6815TR-ND; Part Number (none) -> 0878325623; Price ($) (none) -> 1.56
Changed lines of the file:
@@
 F 1 "Conn_02x07_Odd_Even" H 9950 2276 50  0000 C CNN
 F 2 "uBMS-2:Molex_Milli_Grid_0878325623_TopBottom" H 9900 1850 50  0001 C CNN
-F 3 "~" H 9900 1850 50  0001 C CNN
+F 3 "https://media.digikey.com/pdf/Data%20Sheets/Molex%20PDFs/87832-300_Pkg_Spec.pdf" H 9900 1850 50  0001 C CNN
+F 4 "0878325623" H 9900 1850 50  0001 C CNN "Part Number"
+F 5 "WM6815TR-ND" H 9900 1850 50  0001 C CNN "Digikey Number"
+F 6 "1.56" H 9900 1850 50  0001 C CNN "Price ($)"
+F 7 "Connector Header Surface Mount 14 position 0.079\" (2.00mm)" H 9900 1850 50  0001 C CNN "Comment"
 	1    9900 1850
 	1    0    0    -1

Commit message: Added more part info
- also updated BOM
Parts:
- U11: Comment (none) -> 1 Circuit IC Switch 16:1 160Ohm 24-SSOP; Digikey Number (none) -> 296-9226-2-ND; Part Number (none) -> CD74HC4067SM96; Price ($) (none) -> 0.79
Changed lines of the file:
@@
 F 2 "Package_SO:SSOP-24_5.3x8.2mm_P0.65mm" H 3050 1200 50  0001 C CIN
 F 3 "http://www.ti.com/lit/ds/symlink/cd74hc4067.pdf" H 1650 3050 50  0001 C CNN
+F 4 "CD74HC4067SM96" H 2000 2200 50  0001 C CNN "Part Number"
+F 5 "296-9226-2-ND" H 2000 2200 50  0001 C CNN "Digikey Number"
+F 6 "0.79" H 2000 2200 50  0001 C CNN "Price ($)"
+F 7 "1 Circuit IC Switch 16:1 160Ohm 24-SSOP" H 2000 2200 50  0001 C CNN "Comment"
 	1    2000 2200
 	1    0    0    -1
