File: uBMS-2.sch (KiCad schematic (older format))
At the start: 74 parts, among them J1 Conn_02x03_Counter_Clockwise, J2 Conn_01x02, J3 Conn_01x02, J4 Conn_01x01, Q1 2N7002, Q2 2N7002, Q3 NTD5865NL, U1 LM2576HVS-5, U2 ADS1115IDGS, U3 TLV1117-33, U4 TL431DBV, U5 ESP32-WROOM-32, U6 TSC2012IDT, U7 MCP23017_SS, U8 MCP23008-E_P, U9 VDMG10C0

Commit message: added main power connector
Parts:
- J2, J3: footprint (none) -> uBMS-2:1720430202
Changed lines of the file:
@@
 F 0 "J2" H 1718 4475 50  0000 C CNN
 F 1 "Conn_01x02" H 1718 4566 50  0000 C CNN
-F 2 "" H 1800 4800 50  0001 C CNN
+F 2 "uBMS-2:1720430202" H 1800 4800 50  0001 C CNN
 F 3 "~" H 1800 4800 50  0001 C CNN
 	1    1800 4800
@@
 F 0 "J3" H 1768 5125 50  0000 C CNN
 F 1 "Conn_01x02" H 1768 5216 50  0000 C CNN
-F 2 "" H 1850 5450 50  0001 C CNN
+F 2 "uBMS-2:1720430202" H 1850 5450 50  0001 C CNN
 F 3 "~" H 1850 5450 50  0001 C CNN
 	1    1850 5450
