File: BatteryBalance.sch (KiCad schematic (older format))
At the start: 49 parts, among them J7 Conn_02x07_Counter_Clockwise, Q10 FQD5N20L, Q11 FQD5N20L, Q12 FQD5N20L, Q13 FQD5N20L, Q14 FQD5N20L, Q15 FQD5N20L, Q4 FQD5N20L, Q5 FQD5N20L, Q6 FQD5N20L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

Commit message: Updated balance connector
Parts:
- J7: footprint Connector_PinHeader_2.54mm:PinHeader_2x07_P2.54mm_Vertical -> uBMS-2:CNC-Tech_3020-14-0300-00
Changed lines of the file:
@@
 F 0 "J7" H 10400 3667 50  0000 C CNN
 F 1 "Conn_02x07_Counter_Clockwise" H 10400 3576 50  0000 C CNN
-F 2 "Connector_PinHeader_2.54mm:PinHeader_2x07_P2.54mm_Vertical" H 10350 3150 50  0001 C CNN
+F 2 "uBMS-2:CNC-Tech_3020-14-0300-00" H 10350 3150 50  0001 C CNN
 F 3 "~" H 10350 3150 50  0001 C CNN
 	1    10350 3150

Commit message: Using Molex Milli Grid Connector for 14 pin
Parts:
- J7: footprint uBMS-2:CNC-Tech_3020-14-0300-00 -> uBMS-2:Molex_Milli_Grid_0878325623
Changed lines of the file:
@@
 F 0 "J7" H 10400 3667 50  0000 C CNN
 F 1 "Conn_02x07_Counter_Clockwise" H 10400 3576 50  0000 C CNN
-F 2 "uBMS-2:CNC-Tech_3020-14-0300-00" H 10350 3150 50  0001 C CNN
+F 2 "uBMS-2:Molex_Milli_Grid_0878325623" H 10350 3150 50  0001 C CNN
 F 3 "~" H 10350 3150 50  0001 C CNN
 	1    10350 3150

Commit message: routed and filled a bunch of stuff, so much more to do
Parts:
- removed J7: Conn_02x07_Counter_Clockwise, uBMS-2:Molex_Milli_Grid_0878325623, symbol Connector_Generic:Conn_02x07_Counter_Clockwise
- added J7: Conn_02x07_Odd_Even, uBMS-2:Molex_Milli_Grid_0878325623_TopBottom, symbol Connector_Generic:Conn_02x07_Odd_Even
Connections:
- wire segments 145 -> 146
Changed lines of the file:
@@
 	1    0    0    -1
 $EndComp
+Text Label 10700 2850 0    50   ~ 0
+Cell1_P
 Text Label 10100 2950 2    50   ~ 0
-Cell1_P
+Cell2_P
+Text Label 10700 2950 0    50   ~ 0
+Cell3_P
 Text Label 10100 3050 2    50   ~ 0
-Cell2_P
+Cell4_P
+Text Label 10700 3050 0    50   ~ 0
+Cell5_P
 Text Label 10100 3150 2    50   ~ 0
-Cell3_P
+Cell6_P
+Wire Wire Line
+	9650 2850 10150 2850
+Text Label 10700 3150 0    50   ~ 0
+Cell7_P
 Text Label 10100 3250 2    50   ~ 0
-Cell4_P
-Text Label 10100 3350 2    50   ~ 0
-Cell5_P
-Text Label 10100 3450 2    50   ~ 0
-Cell6_P
-$Comp
-L Connector_Generic:Conn_02x07_Counter_Clockwise J7
-U 1 1 5F78CA28
-P 10350 3150
-F 0 "J7" H 10400 3667 50  0000 C CNN
-F 1 "Conn_02x07_Counter_Clockwise" H 10400 3576 50  0000 C CNN
-F 2 "uBMS-2:Molex_Milli_Grid_0878325623" H 10350 3150 50  0001 C CNN
-F 3 "~" H 10350 3150 50  0001 C CNN
-	1    10350 3150
-	1    0    0    -1
-$EndComp
-Wire Wire Line
-	9650 2850 10150 2850
-Text Label 10700 3450 0    50   ~ 0
-Cell7_P
-Text Label 10700 3350 0    50   ~ 0
 Cell8_P
 Text Label 10700 3250 0    50   ~ 0
 Cell9_P
-Text Label 10700 3150 0    50   ~ 0
+Text Label 10100 3350 2    50   ~ 0
 Cell10_P
-Text Label 10700 3050 0    50   ~ 0
+Text Label 10700 3350 0    50   ~ 0
 Cell11_P
-Text Label 10700 2950 0    50   ~ 0
+Text Label 10100 3450 2    50   ~ 0
 Cell12_P
 Wire Wire Line
@@
 Wire Wire Line
 	10700 2950 10650 2950
-NoConn ~ 10650 2850
 $Comp
 L Device:C C15
@@
 	8500 4850 8450 4850
 Connection ~ 8450 4850
+$Comp
+L Connector_Generic:Conn_02x07_Odd_Even J7
+U 1 1 5F34DEC3
+P 10350 3150
+F 0 "J7" H 10400 3667 50  0000 C CNN
+F 1 "Conn_02x07_Odd_Even" H 10400 3576 50  0000 C CNN
+F 2 "uBMS-2:Molex_Milli_Grid_0878325623_TopBottom" H 10350 3150 50  0001 C CNN
+F 3 "~" H 10350 3150 50  0001 C CNN
+	1    10350 3150
+	1    0    0    -1
+$EndComp
+Wire Wire Line
+	10700 2850 10650 2850
+NoConn ~ 10700 3450
 $EndSCHEMATC

Commit message: Voltage Reg and PTC replacement and balance fet DS caps SCHEMATIC ONLY
- Also added new fields to some of the new parts to make a more complete schematic, I'll slowly be adding this to the other components
- Hopefully the new DC-DC has a MUCH smaller footprint
- Need to fix ESP32 boot issue still
- Need to prepare SMD XT60 Connectors
- Need to remove RGB
- Need to reduce brightness of status LEDs
- Larger NTCs?
- Need to find parts for newly added passives + footprints
- Eventually update the PCB (ah im scared)
- New parts will be going in my ClementsComponents Repo
Parts:
- added C? (x12): 10nF, symbol Device:C_Small
Connections:
- net Cell10_P: now also C?.1, C?.2
- net Cell11_P: now also C?.1, C?.2
- net Cell12_P: now also C?.1
- net Cell1_P: now also C?.1, C?.2
- net Cell2_P: now also C?.1, C?.2
- net Cell3_P: now also C?.1, C?.2
- net Cell4_P: now also C?.1, C?.2
- net Cell5_P: now also C?.1, C?.2
- net Cell6_P: now also C?.1, C?.2
- net Cell7_P: now also C?.1, C?.2
- net Cell8_P: now also C?.1, C?.2
- net Cell9_P: now also C?.1, C?.2
- net GND: now also C?.2

Commit message: Annotated new symbols & Changed Buck Inductor and Freq & Added USB protection diodes
- L1 is now 100uH rated for 1.1A
- Switching freq is now 400kHz
- Need to find proper specced input and output caps
- Does VBus need 3.3v or 5v input?
- R23 is now 71.5k
Parts:
- gave numbers to parts that had none: 12
Changed lines of the file:
@@
 NoConn ~ 10700 3450
 $Comp
-L Device:C_Small C?
+L Device:C_Small C12
 U 1 1 5FF6BD26
 P 2400 1500
-F 0 "C?" H 2492 1546 50  0000 L CNN
+F 0 "C12" H 2492 1546 50  0000 L CNN
 F 1 "10nF" H 2492 1455 50  0000 L CNN
 F 2 "" H 2400 1500 50  0001 C CNN
@@
 Connection ~ 2150 1700
 $Comp
-L Device:C_Small C?
+L Device:C_Small C27
 U 1 1 5FF7CF68
 P 4450 1500
-F 0 "C?" H 4542 1546 50  0000 L CNN
+F 0 "C27" H 4542 1546 50  0000 L CNN
 F 1 "10nF" H 4542 1455 50  0000 L CNN
 F 2 "" H 4450 1500 50  0001 C CNN
@@
 $EndComp
 $Comp
-L Device:C_Small C?
+L Device:C_Small C28
 U 1 1 5FF7D69E
 P 6550 1500
-F 0 "C?" H 6642 1546 50  0000 L CNN
+F 0 "C28" H 6642 1546 50  0000 L CNN
 F 1 "10nF" H 6642 1455 50  0000 L CNN
 F 2 "" H 6550 1500 50  0001 C CNN
@@
 $EndComp
 $Comp
-L Device:C_Small C?
+L Device:C_Small C29
 U 1 1 5FF7DC64
 P 8650 1500
-F 0 "C?" H 8742 1546 50  0000 L CNN
+F 0 "C29" H 8742 1546 50  0000 L CNN
 F 1 "10nF" H 8742 1455 50  0000 L CNN
 F 2 "" H 8650 1500 50  0001 C CNN
@@
 $EndComp
 $Comp
-L Device:C_Small C?
+L Device:C_Small C30
 U 1 1 5FF7E0BA
 P 2350 3000
-F 0 "C?" H 2442 3046 50  0000 L CNN
+F 0 "C30" H 2442 3046 50  0000 L CNN
 F 1 "10nF" H 2442 2955 50  0000 L CNN
 F 2 "" H 2350 3000 50  0001 C CNN
@@
 $EndComp
 $Comp
-L Device:C_Small C?
+L Device:C_Small C31
 U 1 1 5FF7E835
 P 4450 3000
-F 0 "C?" H 4542 3046 50  0000 L CNN
+F 0 "C31" H 4542 3046 50  0000 L CNN
 F 1 "10nF" H 4542 2955 50  0000 L CNN
 F 2 "" H 4450 3000 50  0001 C CNN
@@
 $EndComp
 $Comp
-L Device:C_Small C?
+L Device:C_Small C32
 U 1 1 5FF7ED5A
 P 6550 3000
-F 0 "C?" H 6642 3046 50  0000 L CNN
+F 0 "C32" H 6642 3046 50  0000 L CNN
 F 1 "10nF" H 6642 2955 50  0000 L CNN
 F 2 "" H 6550 3000 50  0001 C CNN
@@
 $EndComp
 $Comp
-L Device:C_Small C?
+L Device:C_Small C33
 U 1 1 5FF7F434
 P 8650 3000
-F 0 "C?" H 8742 3046 50  0000 L CNN
+F 0 "C33" H 8742 3046 50  0000 L CNN
 F 1 "10nF" H 8742 2955 50  0000 L CNN
 F 2 "" H 8650 3000 50  0001 C CNN
@@
 $EndComp
 $Comp
-L Device:C_Small C?
+L Device:C_Small C34
 U 1 1 5FF7F9CC
 P 2350 4500
-F 0 "C?" H 2442 4546 50  0000 L CNN
+F 0 "C34" H 2442 4546 50  0000 L CNN
 F 1 "10nF" H 2442 4455 50  0000 L CNN
 F 2 "" H 2350 4500 50  0001 C CNN
@@
 $EndComp
 $Comp
-L Device:C_Small C?
+L Device:C_Small C35
 U 1 1 5FF802CE
 P 4450 4500
-F 0 "C?" H 4542 4546 50  0000 L CNN
+F 0 "C35" H 4542 4546 50  0000 L CNN
 F 1 "10nF" H 4542 4455 50  0000 L CNN
 F 2 "" H 4450 4500 50  0001 C CNN
@@
 $EndComp
 $Comp
-L Device:C_Small C?
+L Device:C_Small C36
 U 1 1 5FF80C2C
 P 6550 4500
-F 0 "C?" H 6642 4546 50  0000 L CNN
+F 0 "C36" H 6642 4546 50  0000 L CNN
 F 1 "10nF" H 6642 4455 50  0000 L CNN
 F 2 "" H 6550 4500 50  0001 C CNN
@@
 $EndComp
 $Comp
-L Device:C_Small C?
+L Device:C_Small C37
 U 1 1 5FF8110C
 P 8650 4500
-F 0 "C?" H 8742 4546 50  0000 L CNN
+F 0 "C37" H 8742 4546 50  0000 L CNN
 F 1 "10nF" H 8742 4455 50  0000 L CNN
 F 2 "" H 8650 4500 50  0001 C CNN

Commit message: Updated all the caps (I think) mostly changed to 0805
- Added 0603 footprints to new resistors which is slightly different from the old 0603 resistors for some reason???
- Annotated the schematic
- Still need to do the inductor oof
Parts:
- removed C18, C19, C23, C24, C25: 10nF, Capacitor_SMD:C_1206_3216Metric, symbol Device:C
- removed C27, C28, C32, C33, C34: 10nF, symbol Device:C_Small
- added C18, C19, C23, C24, C25: 10nF, Capacitor_SMD:C_0805_2012Metric, symbol Device:C_Small
- added C27, C28, C32, C33, C34: 10nF, Capacitor_SMD:C_0805_2012Metric, symbol Device:C
- C12, C29, C30, C31, C35, C36, C37: footprint (none) -> Capacitor_SMD:C_0805_2012Metric; Comment (none) -> 10000pF ±5% 50V Ceramic Capacitor X7R 0805 (2012 Metric); Digikey Number (none) -> 399-17616-2-ND; Part Number (none) -> C0805C103J5RAC7210; Price ($) (none) -> 0.1
- C15, C16, C17, C20, C21, C22, C26: footprint Capacitor_SMD:C_1206_3216Metric -> Capacitor_SMD:C_0805_2012Metric; Comment (none) -> 10000pF ±5% 50V Ceramic Capacitor X7R 0805 (2012 Metric); Digikey Number (none) -> 399-17616-2-ND; Part Number (none) -> C0805C103J5RAC7210; Price ($) (none) -> 0.1
Connections:
- net Bal_PWM_10: now also C22.2
- net Bal_PWM_11: now also C28.2
- net Bal_PWM_12: now also C34.2; no longer C26.2
- net Bal_PWM_2: now also C20.2; no longer C16.2
- net Bal_PWM_3: now also C26.2; no longer C17.2
- net Bal_PWM_4: now also C32.2
- net Bal_PWM_5: now also C16.2
- net Bal_PWM_6: now also C21.2; no longer C20.2
- net Bal_PWM_7: now also C27.2; no longer C21.2
- net Bal_PWM_8: now also C33.2; no longer C22.2
- net Bal_PWM_9: now also C17.2
- net Cell10_P: now also C31.2, C25.1; no longer C35.1, C36.2
- net Cell11_P: now also C31.1; no longer C36.1
- net Cell1_P: now also C23.2
- net Cell2_P: now also C29.2, C23.1
- net Cell3_P: now also C29.1, C35.2; no longer C29.2
- net Cell4_P: now also C35.1, C18.2; no longer C29.1, C30.2
- net Cell5_P: now also C18.1, C24.2; no longer C30.1, C31.2
- net Cell6_P: now also C30.2, C24.1; no longer C31.1
- net Cell7_P: now also C30.1, C36.2
- net Cell8_P: now also C36.1, C19.2
- net Cell9_P: now also C19.1, C25.2; no longer C35.2
- net at D10.1 (K), Q5.1 (G), R77.1: now also C20.1; no longer C16.1
- net at D11.1 (K), Q6.1 (G), R78.1: now also C26.1; no longer C17.1
- net at D12.1 (K), Q7.1 (G), R79.1: now also C32.1
- net at D13.1 (K), Q8.1 (G), R80.1: now also C16.1
- net at D14.1 (K), Q9.1 (G), R81.1: now also C21.1; no longer C20.1
- net at D15.1 (K), Q10.1 (G), R82.1: now also C27.1; no longer C21.1
- net at D16.1 (K), Q11.1 (G), R83.1: now also C33.1; no longer C22.1
- net at D17.1 (K), Q12.1 (G), R84.1: now also C17.1
- net at D18.1 (K), Q13.1 (G), R85.1: now also C22.1
- net at D19.1 (K), Q14.1 (G), R86.1: now also C28.1
- net at D20.1 (K), Q15.1 (G), R87.1: now also C34.1; no longer C26.1

Commit message: Reset 0604 resistors to smaller (older?) footprint size
Parts:
- R76, R77, R78, R79, R80, R81, R82, R83, R84, R85, R86, R87: footprint Resistor_SMD:R_0603_1608Metric_Pad1.05x0.95mm_HandSolder -> Resistor_SMD:R_0603_1608Metric_Pad0.98x0.95mm_HandSolder
Changed lines of the file:
@@
 F 0 "R76" H 1350 1750 50  0000 L CNN
 F 1 "100k" H 1250 1650 50  0000 L CNN
-F 2 "Resistor_SMD:R_0603_1608Metric_Pad1.05x0.95mm_HandSolder" V 1430 1700 50  0001 C CNN
+F 2 "Resistor_SMD:R_0603_1608Metric_Pad0.98x0.95mm_HandSolder" V 1430 1700 50  0001 C CNN
 F 3 "~" H 1500 1700 50  0001 C CNN
 	1    1500 1700
@@
 F 0 "R77" H 3450 1750 50  0000 L CNN
 F 1 "100k" H 3350 1650 50  0000 L CNN
-F 2 "Resistor_SMD:R_0603_1608Metric_Pad1.05x0.95mm_HandSolder" V 3530 1700 50  0001 C CNN
+F 2 "Resistor_SMD:R_0603_1608Metric_Pad0.98x0.95mm_HandSolder" V 3530 1700 50  0001 C CNN
 F 3 "~" H 3600 1700 50  0001 C CNN
 	1    3600 1700
@@
 F 0 "R78" H 5550 1750 50  0000 L CNN
 F 1 "100k" H 5450 1650 50  0000 L CNN
-F 2 "Resistor_SMD:R_0603_1608Metric_Pad1.05x0.95mm_HandSolder" V 5630 1700 50  0001 C CNN
+F 2 "Resistor_SMD:R_0603_1608Metric_Pad0.98x0.95mm_HandSolder" V 5630 1700 50  0001 C CNN
 F 3 "~" H 5700 1700 50  0001 C CNN
 	1    5700 1700
@@
 F 0 "R79" H 7650 1750 50  0000 L CNN
 F 1 "100k" H 7550 1650 50  0000 L CNN
-F 2 "Resistor_SMD:R_0603_1608Metric_Pad1.05x0.95mm_HandSolder" V 7730 1700 50  0001 C CNN
+F 2 "Resistor_SMD:R_0603_1608Metric_Pad0.98x0.95mm_HandSolder" V 7730 1700 50  0001 C CNN
 F 3 "~" H 7800 1700 50  0001 C CNN
 	1    7800 1700
@@
 F 0 "R80" H 1350 3250 50  0000 L CNN
 F 1 "100k" H 1250 3150 50  0000 L CNN
-F 2 "Resistor_SMD:R_0603_1608Metric_Pad1.05x0.95mm_HandSolder" V 1430 3200 50  0001 C CNN
+F 2 "Resistor_SMD:R_0603_1608Metric_Pad0.98x0.95mm_HandSolder" V 1430 3200 50  0001 C CNN
 F 3 "~" H 1500 3200 50  0001 C CNN
 	1    1500 3200
@@
 F 0 "R81" H 3450 3250 50  0000 L CNN
 F 1 "100k" H 3350 3150 50  0000 L CNN
-F 2 "Resistor_SMD:R_0603_1608Metric_Pad1.05x0.95mm_HandSolder" V 3530 3200 50  0001 C CNN
+F 2 "Resistor_SMD:R_0603_1608Metric_Pad0.98x0.95mm_HandSolder" V 3530 3200 50  0001 C CNN
 F 3 "~" H 3600 3200 50  0001 C CNN
 	1    3600 3200
@@
 F 0 "R82" H 5550 3250 50  0000 L CNN
 F 1 "100k" H 5450 3150 50  0000 L CNN
-F 2 "Resistor_SMD:R_0603_1608Metric_Pad1.05x0.95mm_HandSolder" V 5630 3200 50  0001 C CNN
+F 2 "Resistor_SMD:R_0603_1608Metric_Pad0.98x0.95mm_HandSolder" V 5630 3200 50  0001 C CNN
 F 3 "~" H 5700 3200 50  0001 C CNN
 	1    5700 3200
@@
 F 0 "R83" H 7650 3250 50  0000 L CNN
 F 1 "100k" H 7550 3150 50  0000 L CNN
-F 2 "Resistor_SMD:R_0603_1608Metric_Pad1.05x0.95mm_HandSolder" V 7730 3200 50  0001 C CNN
+F 2 "Resistor_SMD:R_0603_1608Metric_Pad0.98x0.95mm_HandSolder" V 7730 3200 50  0001 C CNN
 F 3 "~" H 7800 3200 50  0001 C CNN
 	1    7800 3200
@@
 F 0 "R84" H 1350 4750 50  0000 L CNN
 F 1 "100k" H 1250 4650 50  0000 L CNN
-F 2 "Resistor_SMD:R_0603_1608Metric_Pad1.05x0.95mm_HandSolder" V 1430 4700 50  0001 C CNN
+F 2 "Resistor_SMD:R_0603_1608Metric_Pad0.98x0.95mm_HandSolder" V 1430 4700 50  0001 C CNN
 F 3 "~" H 1500 4700 50  0001 C CNN
 	1    1500 4700
@@
 F 0 "R85" H 3450 4750 50  0000 L CNN
 F 1 "100k" H 3350 4650 50  0000 L CNN
-F 2 "Resistor_SMD:R_0603_1608Metric_Pad1.05x0.95mm_HandSolder" V 3530 4700 50  0001 C CNN
+F 2 "Resistor_SMD:R_0603_1608Metric_Pad0.98x0.95mm_HandSolder" V 3530 4700 50  0001 C CNN
 F 3 "~" H 3600 4700 50  0001 C CNN
 	1    3600 4700
@@
 F 0 "R86" H 5550 4750 50  0000 L CNN
 F 1 "100k" H 5450 4650 50  0000 L CNN
-F 2 "Resistor_SMD:R_0603_1608Metric_Pad1.05x0.95mm_HandSolder" V 5630 4700 50  0001 C CNN
+F 2 "Resistor_SMD:R_0603_1608Metric_Pad0.98x0.95mm_HandSolder" V 5630 4700 50  0001 C CNN
 F 3 "~" H 5700 4700 50  0001 C CNN
 	1    5700 4700
@@
 F 0 "R87" H 7650 4750 50  0000 L CNN
 F 1 "100k" H 7550 4650 50  0000 L CNN
-F 2 "Resistor_SMD:R_0603_1608Metric_Pad1.05x0.95mm_HandSolder" V 7730 4700 50  0001 C CNN
+F 2 "Resistor_SMD:R_0603_1608Metric_Pad0.98x0.95mm_HandSolder" V 7730 4700 50  0001 C CNN
 F 3 "~" H 7800 4700 50  0001 C CNN
 	1    7800 4700

Commit message: Updated some properties and generated BOM with KiBOM
Parts:
- J7: Comment (none) -> Connector Header Surface Mount 14 position 0.079\" (2.00mm); Digikey Number (none) -> WM6815TR-ND; Part Number (none) -> 0878325623; Price ($) (none) -> 1.56
- Q10, Q11, Q12, Q13, Q14, Q15, Q4, Q5, Q6, Q7, Q8, Q9: Comment (none) -> N-Channel 200V 3.8A (Tc) 2.5W (Ta), 37W (Tc) Surface Mount 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; Digikey Number (none) -> FQD5N20LTMTR-ND; Part Number (none) -> FQD5N20LTM; Price ($) (none) -> 0.59
Changed lines of the file:
@@
 F 2 "Package_TO_SOT_SMD:TO-252-2" H 2850 1450 50  0001 C CNN
 F 3 "https://www.mouser.com/datasheet/2/149/FQD5N20L-266424.pdf" H 2150 1500 50  0001 C CNN
+F 4 "FQD5N20LTM" H 2150 1500 50  0001 C CNN "Part Number"
+F 5 "FQD5N20LTMTR-ND" H 2150 1500 50  0001 C CNN "Digikey Number"
+F 6 "0.59" H 2150 1500 50  0001 C CNN "Price ($)"
+F 7 "N-Channel 200V 3.8A (Tc) 2.5W (Ta), 37W (Tc) Surface Mount D-Pak" H 2150 1500 50  0001 C CNN "Comment"
 	1    2150 1500
 	1    0    0    -1
@@
 F 2 "Package_TO_SOT_SMD:TO-252-2" H 4950 1450 50  0001 C CNN
 F 3 "https://www.mouser.com/datasheet/2/149/FQD5N20L-266424.pdf" H 4250 1500 50  0001 C CNN
+F 4 "FQD5N20LTM" H 4250 1500 50  0001 C CNN "Part Number"
+F 5 "FQD5N20LTMTR-ND" H 4250 1500 50  0001 C CNN "Digikey Number"
+F 6 "0.59" H 4250 1500 50  0001 C CNN "Price ($)"
+F 7 "N-Channel 200V 3.8A (Tc) 2.5W (Ta), 37W (Tc) Surface Mount D-Pak" H 4250 1500 50  0001 C CNN "Comment"
 	1    4250 1500
 	1    0    0    -1
@@
 F 2 "Package_TO_SOT_SMD:TO-252-2" H 7050 1450 50  0001 C CNN
 F 3 "https://www.mouser.com/datasheet/2/149/FQD5N20L-266424.pdf" H 6350 1500 50  0001 C CNN
+F 4 "FQD5N20LTM" H 6350 1500 50  0001 C CNN "Part Number"
+F 5 "FQD5N20LTMTR-ND" H 6350 1500 50  0001 C CNN "Digikey Number"
+F 6 "0.59" H 6350 1500 50  0001 C CNN "Price ($)"
+F 7 "N-Channel 200V 3.8A (Tc) 2.5W (Ta), 37W (Tc) Surface Mount D-Pak" H 6350 1500 50  0001 C CNN "Comment"
 	1    6350 1500
 	1    0    0    -1
@@
 F 2 "Package_TO_SOT_SMD:TO-252-2" H 9150 1450 50  0001 C CNN
 F 3 "https://www.mouser.com/datasheet/2/149/FQD5N20L-266424.pdf" H 8450 1500 50  0001 C CNN
+F 4 "FQD5N20LTM" H 8450 1500 50  0001 C CNN "Part Number"
+F 5 "FQD5N20LTMTR-ND" H 8450 1500 50  0001 C CNN "Digikey Number"
+F 6 "0.59" H 8450 1500 50  0001 C CNN "Price ($)"
+F 7 "N-Channel 200V 3.8A (Tc) 2.5W (Ta), 37W (Tc) Surface Mount D-Pak" H 8450 1500 50  0001 C CNN "Comment"
 	1    8450 1500
 	1    0    0    -1
@@
 F 2 "Package_TO_SOT_SMD:TO-252-2" H 2850 2950 50  0001 C CNN
 F 3 "https://www.mouser.com/datasheet/2/149/FQD5N20L-266424.pdf" H 2150 3000 50  0001 C CNN
+F 4 "FQD5N20LTM" H 2150 3000 50  0001 C CNN "Part Number"
+F 5 "FQD5N20LTMTR-ND" H 2150 3000 50  0001 C CNN "Digikey Number"
+F 6 "0.59" H 2150 3000 50  0001 C CNN "Price ($)"
+F 7 "N-Channel 200V 3.8A (Tc) 2.5W (Ta), 37W (Tc) Surface Mount D-Pak" H 2150 3000 50  0001 C CNN "Comment"
 	1    2150 3000
 	1    0    0    -1
@@
 F 2 "Package_TO_SOT_SMD:TO-252-2" H 4950 2950 50  0001 C CNN
 F 3 "https://www.mouser.com/datasheet/2/149/FQD5N20L-266424.pdf" H 4250 3000 50  0001 C CNN
+F 4 "FQD5N20LTM" H 4250 3000 50  0001 C CNN "Part Number"
+F 5 "FQD5N20LTMTR-ND" H 4250 3000 50  0001 C CNN "Digikey Number"
+F 6 "0.59" H 4250 3000 50  0001 C CNN "Price ($)"
+F 7 "N-Channel 200V 3.8A (Tc) 2.5W (Ta), 37W (Tc) Surface Mount D-Pak" H 4250 3000 50  0001 C CNN "Comment"
 	1    4250 3000
 	1    0    0    -1
@@
 F 2 "Package_TO_SOT_SMD:TO-252-2" H 7050 2950 50  0001 C CNN
 F 3 "https://www.mouser.com/datasheet/2/149/FQD5N20L-266424.pdf" H 6350 3000 50  0001 C CNN
+F 4 "FQD5N20LTM" H 6350 3000 50  0001 C CNN "Part Number"
+F 5 "FQD5N20LTMTR-ND" H 6350 3000 50  0001 C CNN "Digikey Number"
+F 6 "0.59" H 6350 3000 50  0001 C CNN "Price ($)"
+F 7 "N-Channel 200V 3.8A (Tc) 2.5W (Ta), 37W (Tc) Surface Mount D-Pak" H 6350 3000 50  0001 C CNN "Comment"
 	1    6350 3000
 	1    0    0    -1
@@
 F 2 "Package_TO_SOT_SMD:TO-252-2" H 9150 2950 50  0001 C CNN
 F 3 "https://www.mouser.com/datasheet/2/149/FQD5N20L-266424.pdf" H 8450 3000 50  0001 C CNN
+F 4 "FQD5N20LTM" H 8450 3000 50  0001 C CNN "Part Number"
+F 5 "FQD5N20LTMTR-ND" H 8450 3000 50  0001 C CNN "Digikey Number"
+F 6 "0.59" H 8450 3000 50  0001 C CNN "Price ($)"
+F 7 "N-Channel 200V 3.8A (Tc) 2.5W (Ta), 37W (Tc) Surface Mount D-Pak" H 8450 3000 50  0001 C CNN "Comment"
 	1    8450 3000
 	1    0    0    -1
@@
 F 2 "Package_TO_SOT_SMD:TO-252-2" H 2850 4450 50  0001 C CNN
 F 3 "https://www.mouser.com/datasheet/2/149/FQD5N20L-266424.pdf" H 2150 4500 50  0001 C CNN
+F 4 "FQD5N20LTM" H 2150 4500 50  0001 C CNN "Part Number"
+F 5 "FQD5N20LTMTR-ND" H 2150 4500 50  0001 C CNN "Digikey Number"
+F 6 "0.59" H 2150 4500 50  0001 C CNN "Price ($)"
+F 7 "N-Channel 200V 3.8A (Tc) 2.5W (Ta), 37W (Tc) Surface Mount D-Pak" H 2150 4500 50  0001 C CNN "Comment"
 	1    2150 4500
 	1    0    0    -1
@@
 F 2 "Package_TO_SOT_SMD:TO-252-2" H 4950 4450 50  0001 C CNN
 F 3 "https://www.mouser.com/datasheet/2/149/FQD5N20L-266424.pdf" H 4250 4500 50  0001 C CNN
+F 4 "FQD5N20LTM" H 4250 4500 50  0001 C CNN "Part Number"
+F 5 "FQD5N20LTMTR-ND" H 4250 4500 50  0001 C CNN "Digikey Number"
+F 6 "0.59" H 4250 4500 50  0001 C CNN "Price ($)"
+F 7 "N-Channel 200V 3.8A (Tc) 2.5W (Ta), 37W (Tc) Surface Mount D-Pak" H 4250 4500 50  0001 C CNN "Comment"
 	1    4250 4500
 	1    0    0    -1
@@
 	4250 4300 4250 4150
 $Comp
-L uBMS-Parts:FQD5N20L Q14
-U 1 1 5F7BAE82
-P 6350 4500
-F 0 "Q14" H 6400 4350 50  0000 L CNN
-F 1 "FQD5N20L" H 5850 4650 50  0000 L CNN
-F 2 "Package_TO_SOT_SMD:TO-252-2" H 7050 4450 50  0001 C CNN
-F 3 "https://www.mouser.com/datasheet/2/149/FQD5N20L-266424.pdf" H 6350 4500 50  0001 C CNN
-	1    6350 4500
-	1    0    0    -1
-$EndComp
-$Comp
 L Device:R R86
 U 1 1 5F7BAE88
@@
 Text Label 6350 4150 0    50   ~ 0
 Cell11_P
-Wire Wire Line
-	6350 4300 6350 4150
 $Comp
 L uBMS-Parts:FQD5N20L Q15
@@
 F 2 "Package_TO_SOT_SMD:TO-252-2" H 9150 4450 50  0001 C CNN
 F 3 "https://www.mouser.com/datasheet/2/149/FQD5N20L-266424.pdf" H 8450 4500 50  0001 C CNN
+F 4 "FQD5N20LTM" H 8450 4500 50  0001 C CNN "Part Number"
+F 5 "FQD5N20LTMTR-ND" H 8450 4500 50  0001 C CNN "Digikey Number"
+F 6 "0.59" H 8450 4500 50  0001 C CNN "Price ($)"
+F 7 "N-Channel 200V 3.8A (Tc) 2.5W (Ta), 37W (Tc) Surface Mount D-Pak" H 8450 4500 50  0001 C CNN "Comment"
 	1    8450 4500
 	1    0    0    -1
@@
 F 1 "Conn_02x07_Odd_Even" H 10400 3576 50  0000 C CNN
 F 2 "uBMS-2:Molex_Milli_Grid_0878325623_TopBottom" H 10350 3150 50  0001 C CNN
-F 3 "~" H 10350 3150 50  0001 C CNN
+F 3 "https://media.digikey.com/pdf/Data%20Sheets/Molex%20PDFs/87832-300_Pkg_Spec.pdf" H 10350 3150 50  0001 C CNN
+F 4 "0878325623" H 10350 3150 50  0001 C CNN "Part Number"
+F 5 "WM6815TR-ND" H 10350 3150 50  0001 C CNN "Digikey Number"
+F 6 "1.56" H 10350 3150 50  0001 C CNN "Price ($)"
+F 7 "Connector Header Surface Mount 14 position 0.079\" (2.00mm)" H 10350 3150 50  0001 C CNN "Comment"
 	1    10350 3150
 	1    0    0    -1
@@
 Wire Wire Line
 	6550 4300 6350 4300
-Connection ~ 6350 4300
 Wire Wire Line
 	6550 4600 6550 4700
 Wire Wire Line
 	6550 4700 6350 4700
-Connection ~ 6350 4700
 Wire Wire Line
 	8650 4400 8650 4300
@@
 	1    0    0    -1
 $EndComp
+Connection ~ 6350 4700
+Connection ~ 6350 4300
+Wire Wire Line
+	6350 4300 6350 4150
+$Comp
+L uBMS-Parts:FQD5N20L Q14
+U 1 1 5F7BAE82
+P 6350 4500
+F 0 "Q14" H 6400 4350 50  0000 L CNN
+F 1 "FQD5N20L" H 5850 4650 50  0000 L CNN
+F 2 "Package_TO_SOT_SMD:TO-252-2" H 7050 4450 50  0001 C CNN
+F 3 "https://www.mouser.com/datasheet/2/149/FQD5N20L-266424.pdf" H 6350 4500 50  0001 C CNN
+F 4 "FQD5N20LTM" H 6350 4500 50  0001 C CNN "Part Number"
+F 5 "FQD5N20LTMTR-ND" H 6350 4500 50  0001 C CNN "Digikey Number"
+F 6 "0.59" H 6350 4500 50  0001 C CNN "Price ($)"
+F 7 "N-Channel 200V 3.8A (Tc) 2.5W (Ta), 37W (Tc) Surface Mount D-Pak" H 6350 4500 50  0001 C CNN "Comment"
+	1    6350 4500
+	1    0    0    -1
+$EndComp
