File: BatteryBalance.kicad_sch (KiCad schematic)
At the start: 61 parts, among them J7 Conn_02x07_Odd_Even, Q10 FQD5N20L, Q11 FQD5N20L, Q12 FQD5N20L, Q13 FQD5N20L, Q14 FQD5N20L, Q15 FQD5N20L, Q4 FQD5N20L, Q5 FQD5N20L, Q6 FQD5N20L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

Commit message: More schematic updates
Parts:
- C12, C15, C16, C17, C18, C19, C20, C21, C22, C23, C24, C25, C26, C27, C28, C29, C30, C31, C32, C33, C34, C35, C36, C37: footprint Capacitor_SMD:C_0805_2012Metric -> Capacitor_SMD:C_0402_1005Metric
- R76, R77, R78, R79, R80, R81, R82, R83, R84, R85, R86, R87: footprint Resistor_SMD:R_0603_1608Metric_Pad0.98x0.95mm_HandSolder -> Resistor_SMD:R_0402_1005Metric

Commit message: Updated all of component values
Parts:
- C12, C15, C16, C17, C18, C19, C20, C21, C22, C23, C24, C25, C26, C27, C28, C29, C30, C31, C32, C33, C34, C35, C36, C37: Comment 10000pF ±5% 50V Ceramic Capacitor X7R 0805 (2012 Metric) -> 10000 pF ±10% 50V Ceramic Capacitor X7R 0402 (1005 Metric); Digikey Number 399-17616-2-ND -> 490-4762-1-ND; Part Number C0805C103J5RAC7210 -> GCM155R71H103KA55D
- D10, D11, D12, D13, D14, D15, D16, D17, D18, D19, D20, D9: footprint Diode_SMD:D_0603_1608Metric_Pad1.05x0.95mm_HandSolder -> Diode_SMD:D_0402_1005Metric; Comment (none) -> Diode Standard 75 V 150mA Surface Mount 0402/SOD-923F; Digikey Number (none) -> 641-1287-1-ND; Part Number (none) -> CDSQR4148; Price ($) (none) -> 0.4
- R76, R77, R78, R79, R80, R81, R82, R83, R84, R85, R86, R87: Comment (none) -> 100 kOhms ±1% 0.063W, 1/16W Chip Resistor 0402 (1005 Metric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; Digikey Number (none) -> 311-100KLRCT-ND; Part Number (none) -> RC0402FR-07100KL; Price ($) (none) -> 0.1

Commit message: More Layout!
Parts:
- D10, D11, D12, D13, D14, D15, D16, D17, D18, D19, D20, D9: footprint Diode_SMD:D_0402_1005Metric -> Diode_SMD:D_1206_3216Metric; symbol Device:D -> Device:D_Schottky; Comment Diode Standard 75 V 150mA Surface Mount 0402/SOD-923F -> Diode Schottky 20 V 1A Surface Mount 1206 (3216 Metric); Digikey Number 641-1287-1-ND -> 478-7803-1-ND; Part Number CDSQR4148 -> SD1206S020S1R0; Price ($) 0.4 -> 0.42
- R76, R77, R78, R79, R80, R81, R82, R83, R84, R85, R86, R87: footprint Resistor_SMD:R_0402_1005Metric -> Resistor_SMD:R_1206_3216Metric; Comment 100 kOhms ±1% 0.063W, 1/16W Chip Resistor 0402 (1005 Metric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 -> 100 kOhms ±1% 0.25W, 1/4W Chip Resistor 1206 (3216 Metric) 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; Digikey Number 311-100KLRCT-ND -> 13-RC1206FR-13100KLCT-ND; Part Number RC0402FR-07100KL -> RC1206FR-13100KL
Connections:
- net Cell10_P: now also J7.12 (Pin_12); no longer J7.11 (Pin_11)
- net Cell11_P: now also J7.14 (Pin_14); no longer J7.12 (Pin_12)
- net Cell1_P: now also J7.1 (Pin_1); no longer J7.2 (Pin_2)
- net Cell2_P: now also J7.2 (Pin_2); no longer J7.3 (Pin_3)
- net GND: now also J7.3 (Pin_3); no longer J7.1 (Pin_1)
