File: tempmux.kicad_sch (KiCad schematic)
At the start: 23 parts, among them J6 Conn_02x07_Odd_Even, U11 CD74HC4067SM

Commit message: More schematic updates
Parts:
- C14: footprint Capacitor_SMD:C_0805_2012Metric -> Capacitor_SMD:C_0402_1005Metric
- R60, R61, R62, R63, R64, R65, R66, R67, R68, R69, R70, R71, R72, R73, R74, R75: footprint Resistor_SMD:R_0603_1608Metric_Pad0.98x0.95mm_HandSolder -> Resistor_SMD:R_0402_1005Metric
- TH1, TH2, TH3, TH4: footprint Resistor_SMD:R_0201_0603Metric -> Resistor_SMD:R_0402_1005Metric
Changed lines of the file:
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@@
       (effects (font (size 1.27 1.27)) (justify left))
     )
-    (property "Footprint" "Resistor_SMD:R_0201_0603Metric" (id 2) (at 127 96.52 0)
+    (property "Footprint" "Resistor_SMD:R_0402_1005Metric" (id 2) (at 127 96.52 0)
       (effects (font (size 1.27 1.27)) hide)
     )
@@
       (effects (font (size 1.27 1.27)) (justify left))
     )
-    (property "Footprint" "Resistor_SMD:R_0603_1608Metric_Pad0.98x0.95mm_HandSolder" (id 2) (at 125.222 107.95 90)
+    (property "Footprint" "Resistor_SMD:R_0402_1005Metric" (id 2) (at 125.222 107.95 90)
       (effects (font (size 1.27 1.27)) hide)
     )
@@
       (effects (font (size 1.27 1.27)) (justify left))
     )
-    (property "Footprint" "Resistor_SMD:R_0201_0603Metric" (id 2) (at 152.4 96.52 0)
+    (property "Footprint" "Resistor_SMD:R_0402_1005Metric" (id 2) (at 152.4 96.52 0)
       (effects (font (size 1.27 1.27)) hide)
     )
@@
       (effects (font (size 1.27 1.27)) (justify left))
     )
-    (property "Footprint" "Resistor_SMD:R_0603_1608Metric_Pad0.98x0.95mm_HandSolder" (id 2) (at 150.622 107.95 90)
+    (property "Footprint" "Resistor_SMD:R_0402_1005Metric" (id 2) (at 150.622 107.95 90)
       (effects (font (size 1.27 1.27)) hide)
     )
@@
       (effects (font (size 1.27 1.27)) (justify left))
     )
-    (property "Footprint" "Resistor_SMD:R_0201_0603Metric" (id 2) (at 177.8 96.52 0)
+    (property "Footprint" "Resistor_SMD:R_0402_1005Metric" (id 2) (at 177.8 96.52 0)
       (effects (font (size 1.27 1.27)) hide)
     )
@@
       (effects (font (size 1.27 1.27)) (justify left))
     )
-    (property "Footprint" "Resistor_SMD:R_0603_1608Metric_Pad0.98x0.95mm_HandSolder" (id 2) (at 176.022 107.95 90)
+    (property "Footprint" "Resistor_SMD:R_0402_1005Metric" (id 2) (at 176.022 107.95 90)
       (effects (font (size 1.27 1.27)) hide)
     )
@@
       (effects (font (size 1.27 1.27)) (justify left))
     )
-    (property "Footprint" "Resistor_SMD:R_0201_0603Metric" (id 2) (at 203.2 96.52 0)
+    (property "Footprint" "Resistor_SMD:R_0402_1005Metric" (id 2) (at 203.2 96.52 0)
       (effects (font (size 1.27 1.27)) hide)
     )
@@
       (effects (font (size 1.27 1.27)) (justify left))
     )
-    (property "Footprint" "Resistor_SMD:R_0603_1608Metric_Pad0.98x0.95mm_HandSolder" (id 2) (at 201.422 107.95 90)
+    (property "Footprint" "Resistor_SMD:R_0402_1005Metric" (id 2) (at 201.422 107.95 90)
       (effects (font (size 1.27 1.27)) hide)
     )
@@
       (effects (font (size 1.27 1.27)) (justify left))
     )
-    (property "Footprint" "Resistor_SMD:R_0603_1608Metric_Pad0.98x0.95mm_HandSolder" (id 2) (at 125.222 41.91 90)
+    (property "Footprint" "Resistor_SMD:R_0402_1005Metric" (id 2) (at 125.222 41.91 90)
       (effects (font (size 1.27 1.27)) hide)
     )
@@
       (effects (font (size 1.27 1.27)) (justify left))
     )
-    (property "Footprint" "Resistor_SMD:R_0603_1608Metric_Pad0.98x0.95mm_HandSolder" (id 2) (at 137.922 41.91 90)
+    (property "Footprint" "Resistor_SMD:R_0402_1005Metric" (id 2) (at 137.922 41.91 90)
       (effects (font (size 1.27 1.27)) hide)
     )
@@
       (effects (font (size 1.27 1.27)) (justify left))
     )
-    (property "Footprint" "Resistor_SMD:R_0603_1608Metric_Pad0.98x0.95mm_HandSolder" (id 2) (at 150.622 41.91 90)
+    (property "Footprint" "Resistor_SMD:R_0402_1005Metric" (id 2) (at 150.622 41.91 90)
       (effects (font (size 1.27 1.27)) hide)
     )
@@
       (effects (font (size 1.27 1.27)) (justify left))
     )
-    (property "Footprint" "Resistor_SMD:R_0603_1608Metric_Pad0.98x0.95mm_HandSolder" (id 2) (at 163.322 41.91 90)
+    (property "Footprint" "Resistor_SMD:R_0402_1005Metric" (id 2) (at 163.322 41.91 90)
       (effects (font (size 1.27 1.27)) hide)
     )
@@
       (effects (font (size 1.27 1.27)) (justify left))
     )
-    (property "Footprint" "Resistor_SMD:R_0603_1608Metric_Pad0.98x0.95mm_HandSolder" (id 2) (at 176.022 41.91 90)
+    (property "Footprint" "Resistor_SMD:R_0402_1005Metric" (id 2) (at 176.022 41.91 90)
       (effects (font (size 1.27 1.27)) hide)
     )
@@
       (effects (font (size 1.27 1.27)) (justify left))
     )
-    (property "Footprint" "Resistor_SMD:R_0603_1608Metric_Pad0.98x0.95mm_HandSolder" (id 2) (at 188.722 41.91 90)
+    (property "Footprint" "Resistor_SMD:R_0402_1005Metric" (id 2) (at 188.722 41.91 90)
       (effects (font (size 1.27 1.27)) hide)
     )
@@
       (effects (font (size 1.27 1.27)) (justify left))
     )
-    (property "Footprint" "Resistor_SMD:R_0603_1608Metric_Pad0.98x0.95mm_HandSolder" (id 2) (at 125.222 73.66 90)
+    (property "Footprint" "Resistor_SMD:R_0402_1005Metric" (id 2) (at 125.222 73.66 90)
       (effects (font (size 1.27 1.27)) hide)
     )
@@
       (effects (font (size 1.27 1.27)) (justify left))
     )
-    (property "Footprint" "Resistor_SMD:R_0603_1608Metric_Pad0.98x0.95mm_HandSolder" (id 2) (at 137.922 73.66 90)
+    (property "Footprint" "Resistor_SMD:R_0402_1005Metric" (id 2) (at 137.922 73.66 90)
       (effects (font (size 1.27 1.27)) hide)
     )
@@
       (effects (font (size 1.27 1.27)) (justify left))
     )
-    (property "Footprint" "Resistor_SMD:R_0603_1608Metric_Pad0.98x0.95mm_HandSolder" (id 2) (at 150.622 73.66 90)
+    (property "Footprint" "Resistor_SMD:R_0402_1005Metric" (id 2) (at 150.622 73.66 90)
       (effects (font (size 1.27 1.27)) hide)
     )
@@
       (effects (font (size 1.27 1.27)) (justify left))
     )
-    (property "Footprint" "Resistor_SMD:R_0603_1608Metric_Pad0.98x0.95mm_HandSolder" (id 2) (at 163.322 73.66 90)
+    (property "Footprint" "Resistor_SMD:R_0402_1005Metric" (id 2) (at 163.322 73.66 90)
       (effects (font (size 1.27 1.27)) hide)
     )
@@
       (effects (font (size 1.27 1.27)) (justify left))
     )
-    (property "Footprint" "Resistor_SMD:R_0603_1608Metric_Pad0.98x0.95mm_HandSolder" (id 2) (at 176.022 73.66 90)
+    (property "Footprint" "Resistor_SMD:R_0402_1005Metric" (id 2) (at 176.022 73.66 90)
       (effects (font (size 1.27 1.27)) hide)
     )
@@
       (effects (font (size 1.27 1.27)) (justify left))
     )
-    (property "Footprint" "Resistor_SMD:R_0603_1608Metric_Pad0.98x0.95mm_HandSolder" (id 2) (at 188.722 73.66 90)
+    (property "Footprint" "Resistor_SMD:R_0402_1005Metric" (id 2) (at 188.722 73.66 90)
       (effects (font (size 1.27 1.27)) hide)
     )
@@
       (effects (font (size 1.27 1.27)) (justify left))
     )
-    (property "Footprint" "Capacitor_SMD:C_0805_2012Metric" (id 2) (at 54.61 27.94 0)
-      (effects (font (size 1.27 1.27)) hide)
-    )
+    (property "Footprint" "Capacitor_SMD:C_0402_1005Metric" (id 2) (at 54.61 27.94 0)
+      (effects (font (size 1.27 1.27)) hide)
+    )

Commit message: Updated all of component values
Parts:
- C14: Comment 0.1µF -20%, +80% 16V Ceramic Capacitor Y5V 0805 (2012 Metri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 -> 0.1 µF ±10% 16V Ceramic Capacitor X7R 0402 (1005 Metric); Digikey Number 399-9159-2-ND -> 311-1338-1-ND; Part Number C0805C104Z4VACTU -> CC0402KRX7R7BB104; Price ($) 0.11 -> 0.1
- R60, R61, R62, R63, R64, R65, R66, R67, R68, R69, R70, R71: Comment (none) -> 22 kOhms ±1% 0.063W, 1/16W Chip Resistor 0402 (1005 Metric)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; Digikey Number (none) -> 311-22.0KLRCT-ND; Part Number (none) -> RC0402FR-0722KL; Price ($) (none) -> 0.1
- R72, R73, R74, R75: Comment (none) -> 4.7 kOhms ±1% 0.063W, 1/16W Chip Resistor 0402 (1005 Metric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; Digikey Number (none) -> 311-4.7KLRCT-ND; Part Number (none) -> RC0402FR-074K7L; Price ($) (none) -> 0.1
- TH1, TH2, TH3, TH4: Comment (none) -> THERMISTOR NTC 10KOHM 3380K 0402; Digikey Number (none) -> 445-2550-1-ND; Part Number (none) -> NTCG103JF103FT1; Price ($) (none) -> 0.11

Commit message: More Layout!
Connections:
- net Balance_Temp: now also U11.22 (I9); no longer U11.8 (I1)
- net CellTemp_1: now also U11.16 (I15); no longer U11.23 (I8)
- net CellTemp_10: now also U11.5 (I4); no longer U11.6 (I3)
- net CellTemp_11: now also U11.21 (I10); no longer U11.18 (I13)
- net CellTemp_12: now also U11.4 (I5); no longer U11.7 (I2)
- net CellTemp_2: now also U11.9 (I0); no longer U11.2 (I7)
- net CellTemp_3: now also U11.17 (I14); no longer U11.22 (I9)
- net CellTemp_4: now also U11.8 (I1); no longer U11.3 (I6)
- net CellTemp_5: now also U11.18 (I13); no longer U11.21 (I10)
- net CellTemp_6: now also U11.7 (I2); no longer U11.4 (I5)
- net CellTemp_7: now also U11.19 (I12); no longer U11.20 (I11)
- net CellTemp_8: now also U11.6 (I3); no longer U11.5 (I4)
- net CellTemp_9: now also U11.20 (I11); no longer U11.19 (I12)
- net ESP_Temp: now also U11.23 (I8); no longer U11.16 (I15)
- net Mosfet_Temp: now also U11.3 (I6); no longer U11.9 (I0)
- net Power_Temp: now also U11.2 (I7); no longer U11.17 (I14)
