File: voltmux.kicad_sch (KiCad schematic)
At the start: 32 parts, among them J5 Conn_02x07_Odd_Even, U10 CD74HC4067SM

Commit message: More schematic updates
Parts:
- C13: footprint Capacitor_SMD:C_0805_2012Metric -> Capacitor_SMD:C_0402_1005Metric
- R31, R32, R33, R34, R35, R36, R37, R38, R39, R40, R41, R42, R43, R44, R45, R46, R47, R48, R49, R50, R51, R52, R53, R54, R55, R56, R57, R58, R59: footprint Resistor_SMD:R_0603_1608Metric_Pad0.98x0.95mm_HandSolder -> Resistor_SMD:R_0402_1005Metric
Changed lines of the file:
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@@
       (effects (font (size 1.27 1.27)) (justify left))
     )
-    (property "Footprint" "Resistor_SMD:R_0603_1608Metric_Pad0.98x0.95mm_HandSolder" (id 2) (at 132.842 41.91 90)
+    (property "Footprint" "Resistor_SMD:R_0402_1005Metric" (id 2) (at 132.842 41.91 90)
       (effects (font (size 1.27 1.27)) hide)
     )
@@
       (effects (font (size 1.27 1.27)) (justify left))
     )
-    (property "Footprint" "Resistor_SMD:R_0603_1608Metric_Pad0.98x0.95mm_HandSolder" (id 2) (at 132.842 54.61 90)
+    (property "Footprint" "Resistor_SMD:R_0402_1005Metric" (id 2) (at 132.842 54.61 90)
       (effects (font (size 1.27 1.27)) hide)
     )
@@
       (effects (font (size 1.27 1.27)) (justify left))
     )
-    (property "Footprint" "Resistor_SMD:R_0603_1608Metric_Pad0.98x0.95mm_HandSolder" (id 2) (at 148.082 41.91 90)
+    (property "Footprint" "Resistor_SMD:R_0402_1005Metric" (id 2) (at 148.082 41.91 90)
       (effects (font (size 1.27 1.27)) hide)
     )
@@
       (effects (font (size 1.27 1.27)) (justify left))
     )
-    (property "Footprint" "Resistor_SMD:R_0603_1608Metric_Pad0.98x0.95mm_HandSolder" (id 2) (at 148.082 54.61 90)
+    (property "Footprint" "Resistor_SMD:R_0402_1005Metric" (id 2) (at 148.082 54.61 90)
       (effects (font (size 1.27 1.27)) hide)
     )
@@
       (effects (font (size 1.27 1.27)) (justify left))
     )
-    (property "Footprint" "Resistor_SMD:R_0603_1608Metric_Pad0.98x0.95mm_HandSolder" (id 2) (at 163.322 41.91 90)
+    (property "Footprint" "Resistor_SMD:R_0402_1005Metric" (id 2) (at 163.322 41.91 90)
       (effects (font (size 1.27 1.27)) hide)
     )
@@
       (effects (font (size 1.27 1.27)) (justify left))
     )
-    (property "Footprint" "Resistor_SMD:R_0603_1608Metric_Pad0.98x0.95mm_HandSolder" (id 2) (at 163.322 54.61 90)
+    (property "Footprint" "Resistor_SMD:R_0402_1005Metric" (id 2) (at 163.322 54.61 90)
       (effects (font (size 1.27 1.27)) hide)
     )
@@
       (effects (font (size 1.27 1.27)) (justify left))
     )
-    (property "Footprint" "Resistor_SMD:R_0603_1608Metric_Pad0.98x0.95mm_HandSolder" (id 2) (at 178.562 41.91 90)
+    (property "Footprint" "Resistor_SMD:R_0402_1005Metric" (id 2) (at 178.562 41.91 90)
       (effects (font (size 1.27 1.27)) hide)
     )
@@
       (effects (font (size 1.27 1.27)) (justify left))
     )
-    (property "Footprint" "Resistor_SMD:R_0603_1608Metric_Pad0.98x0.95mm_HandSolder" (id 2) (at 178.562 54.61 90)
+    (property "Footprint" "Resistor_SMD:R_0402_1005Metric" (id 2) (at 178.562 54.61 90)
       (effects (font (size 1.27 1.27)) hide)
     )
@@
       (effects (font (size 1.27 1.27)) (justify left))
     )
-    (property "Footprint" "Resistor_SMD:R_0603_1608Metric_Pad0.98x0.95mm_HandSolder" (id 2) (at 193.802 41.91 90)
+    (property "Footprint" "Resistor_SMD:R_0402_1005Metric" (id 2) (at 193.802 41.91 90)
       (effects (font (size 1.27 1.27)) hide)
     )
@@
       (effects (font (size 1.27 1.27)) (justify left))
     )
-    (property "Footprint" "Resistor_SMD:R_0603_1608Metric_Pad0.98x0.95mm_HandSolder" (id 2) (at 193.802 54.61 90)
+    (property "Footprint" "Resistor_SMD:R_0402_1005Metric" (id 2) (at 193.802 54.61 90)
       (effects (font (size 1.27 1.27)) hide)
     )
@@
       (effects (font (size 1.27 1.27)) (justify left))
     )
-    (property "Footprint" "Resistor_SMD:R_0603_1608Metric_Pad0.98x0.95mm_HandSolder" (id 2) (at 209.042 41.91 90)
+    (property "Footprint" "Resistor_SMD:R_0402_1005Metric" (id 2) (at 209.042 41.91 90)
       (effects (font (size 1.27 1.27)) hide)
     )
@@
       (effects (font (size 1.27 1.27)) (justify left))
     )
-    (property "Footprint" "Resistor_SMD:R_0603_1608Metric_Pad0.98x0.95mm_HandSolder" (id 2) (at 209.042 54.61 90)
+    (property "Footprint" "Resistor_SMD:R_0402_1005Metric" (id 2) (at 209.042 54.61 90)
       (effects (font (size 1.27 1.27)) hide)
     )
@@
       (effects (font (size 1.27 1.27)) (justify left))
     )
-    (property "Footprint" "Resistor_SMD:R_0603_1608Metric_Pad0.98x0.95mm_HandSolder" (id 2) (at 136.652 82.55 90)
+    (property "Footprint" "Resistor_SMD:R_0402_1005Metric" (id 2) (at 136.652 82.55 90)
       (effects (font (size 1.27 1.27)) hide)
     )
@@
       (effects (font (size 1.27 1.27)) (justify left))
     )
-    (property "Footprint" "Resistor_SMD:R_0603_1608Metric_Pad0.98x0.95mm_HandSolder" (id 2) (at 136.652 95.25 90)
+    (property "Footprint" "Resistor_SMD:R_0402_1005Metric" (id 2) (at 136.652 95.25 90)
       (effects (font (size 1.27 1.27)) hide)
     )
@@
       (effects (font (size 1.27 1.27)) (justify left))
     )
-    (property "Footprint" "Resistor_SMD:R_0603_1608Metric_Pad0.98x0.95mm_HandSolder" (id 2) (at 154.432 82.55 90)
+    (property "Footprint" "Resistor_SMD:R_0402_1005Metric" (id 2) (at 154.432 82.55 90)
       (effects (font (size 1.27 1.27)) hide)
     )
@@
       (effects (font (size 1.27 1.27)) (justify left))
     )
-    (property "Footprint" "Resistor_SMD:R_0603_1608Metric_Pad0.98x0.95mm_HandSolder" (id 2) (at 154.432 95.25 90)
+    (property "Footprint" "Resistor_SMD:R_0402_1005Metric" (id 2) (at 154.432 95.25 90)
       (effects (font (size 1.27 1.27)) hide)
     )
@@
       (effects (font (size 1.27 1.27)) (justify left))
     )
-    (property "Footprint" "Resistor_SMD:R_0603_1608Metric_Pad0.98x0.95mm_HandSolder" (id 2) (at 172.212 82.55 90)
+    (property "Footprint" "Resistor_SMD:R_0402_1005Metric" (id 2) (at 172.212 82.55 90)
       (effects (font (size 1.27 1.27)) hide)
     )
@@
       (effects (font (size 1.27 1.27)) (justify left))
     )
-    (property "Footprint" "Resistor_SMD:R_0603_1608Metric_Pad0.98x0.95mm_HandSolder" (id 2) (at 172.212 95.25 90)
+    (property "Footprint" "Resistor_SMD:R_0402_1005Metric" (id 2) (at 172.212 95.25 90)
       (effects (font (size 1.27 1.27)) hide)
     )
@@
       (effects (font (size 1.27 1.27)) (justify left))
     )
-    (property "Footprint" "Resistor_SMD:R_0603_1608Metric_Pad0.98x0.95mm_HandSolder" (id 2) (at 189.992 82.55 90)
+    (property "Footprint" "Resistor_SMD:R_0402_1005Metric" (id 2) (at 189.992 82.55 90)
       (effects (font (size 1.27 1.27)) hide)
     )
@@
       (effects (font (size 1.27 1.27)) (justify left))
     )
-    (property "Footprint" "Resistor_SMD:R_0603_1608Metric_Pad0.98x0.95mm_HandSolder" (id 2) (at 189.992 106.68 90)
+    (property "Footprint" "Resistor_SMD:R_0402_1005Metric" (id 2) (at 189.992 106.68 90)
       (effects (font (size 1.27 1.27)) hide)
     )
@@
       (effects (font (size 1.27 1.27)) (justify left))
     )
-    (property "Footprint" "Resistor_SMD:R_0603_1608Metric_Pad0.98x0.95mm_HandSolder" (id 2) (at 207.772 82.55 90)
+    (property "Footprint" "Resistor_SMD:R_0402_1005Metric" (id 2) (at 207.772 82.55 90)
       (effects (font (size 1.27 1.27)) hide)
     )
@@
       (effects (font (size 1.27 1.27)) (justify left))
     )
-    (property "Footprint" "Resistor_SMD:R_0603_1608Metric_Pad0.98x0.95mm_HandSolder" (id 2) (at 207.772 95.25 90)
+    (property "Footprint" "Resistor_SMD:R_0402_1005Metric" (id 2) (at 207.772 95.25 90)
       (effects (font (size 1.27 1.27)) hide)
     )
@@
       (effects (font (size 1.27 1.27)) (justify left))
     )
-    (property "Footprint" "Resistor_SMD:R_0603_1608Metric_Pad0.98x0.95mm_HandSolder" (id 2) (at 178.562 62.23 90)
+    (property "Footprint" "Resistor_SMD:R_0402_1005Metric" (id 2) (at 178.562 62.23 90)
       (effects (font (size 1.27 1.27)) hide)
     )
@@
       (effects (font (size 1.27 1.27)) (justify left))
     )
-    (property "Footprint" "Resistor_SMD:R_0603_1608Metric_Pad0.98x0.95mm_HandSolder" (id 2) (at 209.042 62.23 90)
+    (property "Footprint" "Resistor_SMD:R_0402_1005Metric" (id 2) (at 209.042 62.23 90)
       (effects (font (size 1.27 1.27)) hide)
     )
@@
       (effects (font (size 1.27 1.27)) (justify left))
     )
-    (property "Footprint" "Resistor_SMD:R_0603_1608Metric_Pad0.98x0.95mm_HandSolder" (id 2) (at 136.652 102.87 90)
+    (property "Footprint" "Resistor_SMD:R_0402_1005Metric" (id 2) (at 136.652 102.87 90)
       (effects (font (size 1.27 1.27)) hide)
     )
@@
       (effects (font (size 1.27 1.27)) (justify left))
     )
-    (property "Footprint" "Resistor_SMD:R_0603_1608Metric_Pad0.98x0.95mm_HandSolder" (id 2) (at 154.432 102.87 90)
+    (property "Footprint" "Resistor_SMD:R_0402_1005Metric" (id 2) (at 154.432 102.87 90)
       (effects (font (size 1.27 1.27)) hide)
     )
@@
       (effects (font (size 1.27 1.27)) (justify left))
     )
-    (property "Footprint" "Resistor_SMD:R_0603_1608Metric_Pad0.98x0.95mm_HandSolder" (id 2) (at 172.212 102.87 90)
+    (property "Footprint" "Resistor_SMD:R_0402_1005Metric" (id 2) (at 172.212 102.87 90)
       (effects (font (size 1.27 1.27)) hide)
     )
@@
       (effects (font (size 1.27 1.27)) (justify left))
     )
-    (property "Footprint" "Resistor_SMD:R_0603_1608Metric_Pad0.98x0.95mm_HandSolder" (id 2) (at 189.992 90.17 90)
+    (property "Footprint" "Resistor_SMD:R_0402_1005Metric" (id 2) (at 189.992 90.17 90)
       (effects (font (size 1.27 1.27)) hide)
     )
@@
       (effects (font (size 1.27 1.27)) (justify left))
     )
-    (property "Footprint" "Resistor_SMD:R_0603_1608Metric_Pad0.98x0.95mm_HandSolder" (id 2) (at 207.772 102.87 90)
+    (property "Footprint" "Resistor_SMD:R_0402_1005Metric" (id 2) (at 207.772 102.87 90)
       (effects (font (size 1.27 1.27)) hide)
     )
@@
       (effects (font (size 1.27 1.27)) (justify left))
     )
-    (property "Footprint" "Capacitor_SMD:C_0805_2012Metric" (id 2) (at 63.5 31.75 0)
-      (effects (font (size 1.27 1.27)) hide)
-    )
+    (property "Footprint" "Capacitor_SMD:C_0402_1005Metric" (id 2) (at 63.5 31.75 0)
+      (effects (font (size 1.27 1.27)) hide)
+    )

Commit message: Updated all of component values
Parts:
- C13: Comment 0.1µF -20%, +80% 16V Ceramic Capacitor Y5V 0805 (2012 Metri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 -> 0.1 µF ±10% 16V Ceramic Capacitor X7R 0402 (1005 Metric); Digikey Number 399-9159-2-ND -> 311-1338-1-ND; Part Number C0805C104Z4VACTU -> CC0402KRX7R7BB104; Price ($) 0.11 -> 0.1
- R31, R37: Comment (none) -> 360 kOhms ±1% 0.063W, 1/16W Chip Resistor 0402 (1005 Metric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; Digikey Number (none) -> 311-360KLRCT-ND; Part Number (none) -> RC0402FR-07360KL; Price ($) (none) -> 0.1
- R32: Comment (none) -> 200 kOhms ±1% 0.063W, 1/16W Chip Resistor 0402 (1005 Metric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; Digikey Number (none) -> 311-200KLRCT-ND; Part Number (none) -> RC0402FR-07200KL; Price ($) (none) -> 0.1
- R33, R48: Comment (none) -> 330 kOhms ±5% 0.063W, 1/16W Chip Resistor 0402 (1005 Metric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; Digikey Number (none) -> 311-330KJRCT-ND; Part Number (none) -> RC0402JR-07330KL; Price ($) (none) -> 0.1
- R34, R35, R46, R49: value 500k -> 499k; Comment (none) -> 499 kOhms ±1% 0.063W, 1/16W Chip Resistor 0402 (1005 Metric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; Digikey Number (none) -> 311-499KLRCT-ND; Part Number (none) -> RC0402FR-07499KL; Price ($) (none) -> 0.1
- R36, R45, R47: Comment (none) -> 560 kOhms ±1% 0.063W, 1/16W Chip Resistor 0402 (1005 Metric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; Digikey Number (none) -> 311-560KLRCT-ND; Part Number (none) -> RC0402FR-07560KL; Price ($) (none) -> 0.1
- R38, R39, R40, R41: Comment (none) -> 100 kOhms ±1% 0.063W, 1/16W Chip Resistor 0402 (1005 Metric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; Digikey Number (none) -> 311-100KLRCT-ND; Part Number (none) -> RC0402FR-07100KL; Price ($) (none) -> 0.1
- R42, R44: Comment (none) -> 47 kOhms ±1% 0.063W, 1/16W Chip Resistor 0402 (1005 Metric)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; Digikey Number (none) -> 311-47.0KLRCT-ND; Part Number (none) -> RC0402FR-0747KL; Price ($) (none) -> 0.1
- R43: value 25k -> 24.9k; Comment (none) -> 24.9 kOhms ±1% 0.063W, 1/16W Chip Resistor 0402 (1005 Metri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; Digikey Number (none) -> 311-24.9KLRCT-ND; Part Number (none) -> RC0402FR-0724K9L; Price ($) (none) -> 0.1
- R50: Comment (none) -> 147 kOhms ±1% 0.063W, 1/16W Chip Resistor 0402 (1005 Metric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; Digikey Number (none) -> YAG2981CT-ND; Part Number (none) -> RC0402FR-07147KL; Price ($) (none) -> 0.1
- R51, R55: Comment (none) -> 39.2 kOhms ±1% 0.063W, 1/16W Chip Resistor 0402 (1005 Metri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; Digikey Number (none) -> 311-39.2KLRCT-ND; Part Number (none) -> RC0402FR-0739K2L; Price ($) (none) -> 0.1
- R52, R53, R54: Comment (none) -> 30 kOhms ±1% 0.063W, 1/16W Chip Resistor 0402 (1005 Metric)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; Digikey Number (none) -> 311-30.0KLRCT-ND; Part Number (none) -> RC0402FR-0730KL; Price ($) (none) -> 0.1
- R56, R57: Comment (none) -> 33.2 kOhms ±1% 0.063W, 1/16W Chip Resistor 0402 (1005 Metri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; Digikey Number (none) -> 311-33.2KLRCT-ND; Part Number (none) -> RC0402FR-0733K2L; Price ($) (none) -> 0.1
- R58: Comment (none) -> 16.2 kOhms ±1% 0.063W, 1/16W Chip Resistor 0402 (1005 Metri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; Digikey Number (none) -> 311-16.2KLRCT-ND; Part Number (none) -> RC0402FR-0716K2L; Price ($) (none) -> 0.1
- R59: Comment (none) -> 47.5 kOhms ±1% 0.063W, 1/16W Chip Resistor 0402 (1005 Metri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; Digikey Number (none) -> 311-47.5KLRCT-ND; Part Number (none) -> RC0402FR-0747K5L; Price ($) (none) -> 0.1

Commit message: More Layout!
Parts:
- added R107: 30k, Resistor_SMD:R_0402_1005Metric, symbol Device:R
Connections:
- net Cell10_Sense: now also U10.22 (I9); no longer U10.21 (I10)
- net Cell11_Sense: now also U10.2 (I7); no longer U10.6 (I3)
- net Cell12_Sense: now also U10.23 (I8); no longer U10.22 (I9)
- net Cell2_Sense: now also U10.8 (I1); no longer U10.23 (I8)
- net Cell3_Sense: now also U10.6 (I3); no longer U10.2 (I7)
- net Cell5_Sense: now also U10.5 (I4); no longer U10.3 (I6)
- net Cell6_Sense: now also U10.20 (I11); no longer U10.8 (I1)
- net Cell8_Sense: now also U10.21 (I10); no longer U10.20 (I11)
- net Cell9_Sense: now also U10.3 (I6); no longer U10.5 (I4)
- net GND: now also J5.14 (Pin_14), R107.2; no longer U10.16 (I15), U10.17 (I14), U10.18 (I13), U10.19 (I12)
- new net: R107.1, U10.16 (I15), U10.17 (I14), U10.18 (I13), U10.19 (I12)
- no-connect marks 1 -> 0
