File: uBMS-2.kicad_sch (KiCad schematic)
At the start: 100 parts, among them J1 DX07S016JA1R1500, J2 XT60PW-M20, J3 XT60PW-M20, Q3 NTD5865NL, SW1 PTS815_SJK_250_SMTR_LFS, SW2 PTS815_SJK_250_SMTR_LFS, SW3 PTS815_SJK_250_SMTR_LFS, U1 ESP32-S2-MINI-1, U13 SN74HC595BRWNR, U2 ADS1115IDGS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

Commit message: ALMOST THERE
Connections:
- net ADC_RDY_3V3: now also U1.38 (IO42); no longer U1.37 (IO41)
- net SER_5V: now also U7.14 (SER); no longer U13.14 (SER)
- net SREG_1_OUT: now also U7.9 (QH'), U8.14 (SER); no longer U13.9 (QH'), U7.14 (SER)
- net SREG_2_OUT: now also U13.14 (SER), U8.9 (QH'); no longer U7.9 (QH'), U8.14 (SER)
- new net UBER_EN: U1.37 (IO41)
- no-connect marks 10 -> 9
Other:
- sheet Level Shifts ports: added UBER_EN; removed none
- moved on the sheet: C40, TP1
